File: a5984_stepper.sch (KiCad schematic (older format))
At the start: 14 parts

Commit message: Possibly finished schematic.
Parts:
- gave numbers to parts that had none: 14

Commit message: Start working on footprint assignments.
Parts:
- C201, C202: footprint (none) -> Capacitors_SMD:C_0805_HandSoldering
- P201: value CONN_01X04 -> MOT; footprint (none) -> Pin_Headers:Pin_Header_Straight_1x04
- R201, R202, R203, R204, R205: footprint (none) -> Resistors_SMD:R_0805_HandSoldering
Changed lines of the file:
@@
 $Descr A4 11693 8268
 encoding utf-8
-Sheet 2 8
+Sheet 5 8
 Title ""
 Date ""
@@
 AR Path="/57A011F0/579F4813" Ref="U401"  Part="1"
 AR Path="/57A0221A/579F4813" Ref="U501"  Part="1"
-F 0 "U201" H 5890 2850 60  0000 C CNN
+F 0 "U301" H 5890 2850 60  0000 C CNN
 F 1 "A5984" H 5630 3670 60  0000 C CNN
-F 2 "" H 5630 3670 60  0000 C CNN
+F 2 "" H 5630 3670 60  0001 C CNN
 F 3 "" H 5630 3670 60  0000 C CNN
 	1    5630 3670
@@
 AR Path="/57A011F0/579F48E9" Ref="C401"  Part="1"
 AR Path="/57A0221A/579F48E9" Ref="C501"  Part="1"
-F 0 "C201" H 5530 2790 50  0000 L CNN
+F 0 "C301" H 5530 2790 50  0000 L CNN
 F 1 "0.1uf" H 5530 2640 50  0000 L CNN
-F 2 "" H 5520 2720 50  0000 C CNN
+F 2 "Capacitors_SMD:C_0805_HandSoldering" H 5520 2720 50  0001 C CNN
 F 3 "" H 5520 2720 50  0000 C CNN
 	1    5520 2720
@@
 AR Path="/57A011F0/579F4A31" Ref="C402"  Part="1"
 AR Path="/57A0221A/579F4A31" Ref="C502"  Part="1"
-F 0 "C202" H 5990 2960 50  0000 L CNN
+F 0 "C302" H 5990 2960 50  0000 L CNN
 F 1 "0.1uf" H 5990 2810 50  0000 L CNN
-F 2 "" H 5980 2890 50  0000 C CNN
+F 2 "Capacitors_SMD:C_0805_HandSoldering" H 5980 2890 50  0001 C CNN
 F 3 "" H 5980 2890 50  0000 C CNN
 	1    5980 2890
@@
 AR Path="/57A011F0/579F5380" Ref="#PWR025"  Part="1"
 AR Path="/57A0221A/579F5380" Ref="#PWR027"  Part="1"
-F 0 "#PWR027" H 6530 2940 50  0001 C CNN
+F 0 "#PWR023" H 6530 2940 50  0001 C CNN
 F 1 "GND" H 6530 3040 50  0000 C CNN
 F 2 "" H 6530 3190 50  0000 C CNN
@@
 AR Path="/57A011F0/579F53B1" Ref="C403"  Part="1"
 AR Path="/57A0221A/579F53B1" Ref="C503"  Part="1"
-F 0 "C203" H 6540 3140 50  0000 L CNN
+F 0 "C303" H 6540 3140 50  0000 L CNN
 F 1 "100uf" H 6540 2990 50  0000 L CNN
-F 2 "" H 6530 3070 50  0000 C CNN
+F 2 "" H 6530 3070 50  0001 C CNN
 F 3 "" H 6530 3070 50  0000 C CNN
 	1    6530 3070
@@
 AR Path="/57A011F0/579F5CC2" Ref="R404"  Part="1"
 AR Path="/57A0221A/579F5CC2" Ref="R504"  Part="1"
-F 0 "R204" H 6440 4290 50  0000 L CNN
+F 0 "R304" H 6440 4290 50  0000 L CNN
 F 1 "0.05" H 6440 4230 50  0000 L CNN
-F 2 "" H 6410 4270 50  0000 C CNN
+F 2 "Resistors_SMD:R_0805_HandSoldering" H 6410 4270 50  0001 C CNN
 F 3 "" H 6410 4270 50  0000 C CNN
 	1    6410 4270
@@
 AR Path="/57A011F0/579F5D70" Ref="R405"  Part="1"
 AR Path="/57A0221A/579F5D70" Ref="R505"  Part="1"
-F 0 "R205" H 6700 4290 50  0000 L CNN
+F 0 "R305" H 6700 4290 50  0000 L CNN
 F 1 "0.05" H 6700 4230 50  0000 L CNN
-F 2 "" H 6670 4270 50  0000 C CNN
+F 2 "Resistors_SMD:R_0805_HandSoldering" H 6670 4270 50  0001 C CNN
 F 3 "" H 6670 4270 50  0000 C CNN
 	1    6670 4270
@@
 AR Path="/57A011F0/579F5F9F" Ref="#PWR026"  Part="1"
 AR Path="/57A0221A/579F5F9F" Ref="#PWR028"  Part="1"
-F 0 "#PWR028" H 6100 4460 50  0001 C CNN
+F 0 "#PWR024" H 6100 4460 50  0001 C CNN
 F 1 "GND" H 6100 4560 50  0000 C CNN
 F 2 "" H 6100 4710 50  0000 C CNN
@@
 AR Path="/57A011F0/579F6126" Ref="P401"  Part="1"
 AR Path="/57A0221A/579F6126" Ref="P501"  Part="1"
-F 0 "P201" H 6530 3950 50  0000 C CNN
-F 1 "CONN_01X04" V 6630 3700 50  0000 C CNN
-F 2 "" H 6530 3700 50  0000 C CNN
+F 0 "P301" H 6530 3950 50  0000 C CNN
+F 1 "MOT" V 6630 3700 50  0000 C CNN
+F 2 "Pin_Headers:Pin_Header_Straight_1x04" H 6530 3700 50  0001 C CNN
 F 3 "" H 6530 3700 50  0000 C CNN
 	1    6530 3700
@@
 AR Path="/57A011F0/579F6BCE" Ref="JP403"  Part="1"
 AR Path="/57A0221A/579F6BCE" Ref="JP503"  Part="1"
-F 0 "JP203" H 4990 3640 50  0000 C CNN
+F 0 "JP303" H 4990 3640 50  0000 C CNN
 F 1 "Jumper_NC_Small" H 5000 3500 50  0001 C CNN
-F 2 "" H 4990 3560 50  0000 C CNN
+F 2 "" H 4990 3560 50  0001 C CNN
 F 3 "" H 4990 3560 50  0000 C CNN
 	1    4990 3560
@@
 AR Path="/57A011F0/579F6D26" Ref="JP402"  Part="1"
 AR Path="/57A0221A/579F6D26" Ref="JP502"  Part="1"
-F 0 "JP202" H 4810 3730 50  0000 C CNN
+F 0 "JP302" H 4810 3730 50  0000 C CNN
 F 1 "Jumper_NC_Small" H 4820 3590 50  0001 C CNN
-F 2 "" H 4810 3650 50  0000 C CNN
+F 2 "" H 4810 3650 50  0001 C CNN
 F 3 "" H 4810 3650 50  0000 C CNN
 	1    4810 3650
@@
 AR Path="/57A011F0/579F6D99" Ref="JP401"  Part="1"
 AR Path="/57A0221A/579F6D99" Ref="JP501"  Part="1"
-F 0 "JP201" H 4640 3820 50  0000 C CNN
+F 0 "JP301" H 4640 3820 50  0000 C CNN
 F 1 "Jumper_NC_Small" H 4650 3680 50  0001 C CNN
-F 2 "" H 4640 3740 50  0000 C CNN
+F 2 "" H 4640 3740 50  0001 C CNN
 F 3 "" H 4640 3740 50  0000 C CNN
 	1    4640 3740
@@
 AR Path="/57A011F0/579F823F" Ref="R402"  Part="1"
 AR Path="/57A0221A/579F823F" Ref="R502"  Part="1"
-F 0 "R202" V 4600 3890 50  0000 L CNN
+F 0 "R302" V 4600 3890 50  0000 L CNN
 F 1 "100k" V 4730 3850 50  0000 L CNN
-F 2 "" H 4660 3930 50  0000 C CNN
+F 2 "Resistors_SMD:R_0805_HandSoldering" H 4660 3930 50  0001 C CNN
 F 3 "" H 4660 3930 50  0000 C CNN
 	1    4660 3930
@@
 AR Path="/57A011F0/579F8AB7" Ref="R403"  Part="1"
 AR Path="/57A0221A/579F8AB7" Ref="R503"  Part="1"
-F 0 "R203" V 4780 3230 50  0000 L CNN
+F 0 "R303" V 4780 3230 50  0000 L CNN
 F 1 "100k" V 4910 3190 50  0000 L CNN
-F 2 "" H 4840 3270 50  0000 C CNN
+F 2 "Resistors_SMD:R_0805_HandSoldering" H 4840 3270 50  0001 C CNN
 F 3 "" H 4840 3270 50  0000 C CNN
 	1    4840 3270
@@
 AR Path="/57A011F0/579FAB17" Ref="RV401"  Part="1"
 AR Path="/57A0221A/579FAB17" Ref="RV501"  Part="1"
-F 0 "RV201" H 4460 4000 50  0000 C CNN
+F 0 "RV301" H 4460 4000 50  0000 C CNN
 F 1 "100k" H 4460 4080 50  0000 C CNN
-F 2 "" H 4460 4080 50  0000 C CNN
+F 2 "" H 4460 4080 50  0001 C CNN
 F 3 "" H 4460 4080 50  0000 C CNN
 	1    4460 4080
@@
 AR Path="/57A011F0/579FAC77" Ref="R401"  Part="1"
 AR Path="/57A0221A/579FAC77" Ref="R501"  Part="1"
-F 0 "R201" H 4490 3850 50  0000 L CNN
+F 0 "R301" H 4490 3850 50  0000 L CNN
 F 1 "20k" H 4490 3790 50  0000 L CNN
-F 2 "" H 4460 3830 50  0000 C CNN
+F 2 "Resistors_SMD:R_0805_HandSoldering" H 4460 3830 50  0001 C CNN
 F 3 "" H 4460 3830 50  0000 C CNN
 	1    4460 3830

Commit message: Finish assigning footprints.
Parts:
- C203: footprint (none) -> Capacitors_SMD:c_elec_6.3x5.8; MPN (none) -> UWT1V101MCL1GS
- JP201, JP202, JP203: footprint (none) -> stmps:MADW__SMD-solder-bridge-narrow
- RV201: footprint (none) -> stmps:BOURNS-TC33X-2
- U201: footprint (none) -> stmps:TSSOP-24_4.4x7.8mm_Pitch0.65mm
Changed lines of the file:
@@
 $Descr A4 11693 8268
 encoding utf-8
-Sheet 5 8
+Sheet 2 8
 Title ""
 Date ""
@@
 AR Path="/57A011F0/579F4813" Ref="U401"  Part="1"
 AR Path="/57A0221A/579F4813" Ref="U501"  Part="1"
-F 0 "U301" H 5890 2850 60  0000 C CNN
+F 0 "U501" H 5890 2850 60  0000 C CNN
 F 1 "A5984" H 5630 3670 60  0000 C CNN
-F 2 "" H 5630 3670 60  0001 C CNN
+F 2 "stmps:TSSOP-24_4.4x7.8mm_Pitch0.65mm" H 5630 3670 60  0001 C CNN
 F 3 "" H 5630 3670 60  0000 C CNN
 	1    5630 3670
@@
 AR Path="/57A011F0/579F48E9" Ref="C401"  Part="1"
 AR Path="/57A0221A/579F48E9" Ref="C501"  Part="1"
-F 0 "C301" H 5530 2790 50  0000 L CNN
+F 0 "C501" H 5530 2790 50  0000 L CNN
 F 1 "0.1uf" H 5530 2640 50  0000 L CNN
 F 2 "Capacitors_SMD:C_0805_HandSoldering" H 5520 2720 50  0001 C CNN
@@
 AR Path="/57A011F0/579F4A31" Ref="C402"  Part="1"
 AR Path="/57A0221A/579F4A31" Ref="C502"  Part="1"
-F 0 "C302" H 5990 2960 50  0000 L CNN
+F 0 "C502" H 5990 2960 50  0000 L CNN
 F 1 "0.1uf" H 5990 2810 50  0000 L CNN
 F 2 "Capacitors_SMD:C_0805_HandSoldering" H 5980 2890 50  0001 C CNN
@@
 +12v
 $Comp
-L GND #PWR021
+L GND #PWR022
 U 1 1 579F5380
 P 6530 3190
-AR Path="/579F3F70/579F5380" Ref="#PWR021"  Part="1"
-AR Path="/57A00526/579F5380" Ref="#PWR023"  Part="1"
-AR Path="/57A011F0/579F5380" Ref="#PWR025"  Part="1"
-AR Path="/57A0221A/579F5380" Ref="#PWR027"  Part="1"
-F 0 "#PWR023" H 6530 2940 50  0001 C CNN
+AR Path="/579F3F70/579F5380" Ref="#PWR022"  Part="1"
+AR Path="/57A00526/579F5380" Ref="#PWR024"  Part="1"
+AR Path="/57A011F0/579F5380" Ref="#PWR026"  Part="1"
+AR Path="/57A0221A/579F5380" Ref="#PWR028"  Part="1"
+F 0 "#PWR028" H 6530 2940 50  0001 C CNN
 F 1 "GND" H 6530 3040 50  0000 C CNN
 F 2 "" H 6530 3190 50  0000 C CNN
@@
 AR Path="/57A011F0/579F53B1" Ref="C403"  Part="1"
 AR Path="/57A0221A/579F53B1" Ref="C503"  Part="1"
-F 0 "C303" H 6540 3140 50  0000 L CNN
+F 0 "C503" H 6540 3140 50  0000 L CNN
 F 1 "100uf" H 6540 2990 50  0000 L CNN
-F 2 "" H 6530 3070 50  0001 C CNN
+F 2 "Capacitors_SMD:c_elec_6.3x5.8" H 6530 3070 50  0001 C CNN
 F 3 "" H 6530 3070 50  0000 C CNN
+F 4 "UWT1V101MCL1GS" H 6530 3070 60  0001 C CNN "MPN"
 	1    6530 3070
 	1    0    0    -1
@@
 AR Path="/57A011F0/579F5CC2" Ref="R404"  Part="1"
 AR Path="/57A0221A/579F5CC2" Ref="R504"  Part="1"
-F 0 "R304" H 6440 4290 50  0000 L CNN
+F 0 "R504" H 6440 4290 50  0000 L CNN
 F 1 "0.05" H 6440 4230 50  0000 L CNN
 F 2 "Resistors_SMD:R_0805_HandSoldering" H 6410 4270 50  0001 C CNN
@@
 AR Path="/57A011F0/579F5D70" Ref="R405"  Part="1"
 AR Path="/57A0221A/579F5D70" Ref="R505"  Part="1"
-F 0 "R305" H 6700 4290 50  0000 L CNN
+F 0 "R505" H 6700 4290 50  0000 L CNN
 F 1 "0.05" H 6700 4230 50  0000 L CNN
 F 2 "Resistors_SMD:R_0805_HandSoldering" H 6670 4270 50  0001 C CNN
@@
 $EndComp
 $Comp
-L GND #PWR022
+L GND #PWR023
 U 1 1 579F5F9F
 P 6100 4710
-AR Path="/579F3F70/579F5F9F" Ref="#PWR022"  Part="1"
-AR Path="/57A00526/579F5F9F" Ref="#PWR024"  Part="1"
-AR Path="/57A011F0/579F5F9F" Ref="#PWR026"  Part="1"
-AR Path="/57A0221A/579F5F9F" Ref="#PWR028"  Part="1"
-F 0 "#PWR024" H 6100 4460 50  0001 C CNN
+AR Path="/579F3F70/579F5F9F" Ref="#PWR023"  Part="1"
+AR Path="/57A00526/579F5F9F" Ref="#PWR025"  Part="1"
+AR Path="/57A011F0/579F5F9F" Ref="#PWR027"  Part="1"
+AR Path="/57A0221A/579F5F9F" Ref="#PWR029"  Part="1"
+F 0 "#PWR029" H 6100 4460 50  0001 C CNN
 F 1 "GND" H 6100 4560 50  0000 C CNN
 F 2 "" H 6100 4710 50  0000 C CNN
@@
 AR Path="/57A011F0/579F6126" Ref="P401"  Part="1"
 AR Path="/57A0221A/579F6126" Ref="P501"  Part="1"
-F 0 "P301" H 6530 3950 50  0000 C CNN
+F 0 "P501" H 6530 3950 50  0000 C CNN
 F 1 "MOT" V 6630 3700 50  0000 C CNN
 F 2 "Pin_Headers:Pin_Header_Straight_1x04" H 6530 3700 50  0001 C CNN
@@
 AR Path="/57A011F0/579F6BCE" Ref="JP403"  Part="1"
 AR Path="/57A0221A/579F6BCE" Ref="JP503"  Part="1"
-F 0 "JP303" H 4990 3640 50  0000 C CNN
+F 0 "JP503" H 4990 3640 50  0000 C CNN
 F 1 "Jumper_NC_Small" H 5000 3500 50  0001 C CNN
-F 2 "" H 4990 3560 50  0001 C CNN
+F 2 "stmps:MADW__SMD-solder-bridge-narrow" H 4990 3560 50  0001 C CNN
 F 3 "" H 4990 3560 50  0000 C CNN
 	1    4990 3560
@@
 AR Path="/57A011F0/579F6D26" Ref="JP402"  Part="1"
 AR Path="/57A0221A/579F6D26" Ref="JP502"  Part="1"
-F 0 "JP302" H 4810 3730 50  0000 C CNN
+F 0 "JP502" H 4810 3730 50  0000 C CNN
 F 1 "Jumper_NC_Small" H 4820 3590 50  0001 C CNN
-F 2 "" H 4810 3650 50  0001 C CNN
+F 2 "stmps:MADW__SMD-solder-bridge-narrow" H 4810 3650 50  0001 C CNN
 F 3 "" H 4810 3650 50  0000 C CNN
 	1    4810 3650
@@
 AR Path="/57A011F0/579F6D99" Ref="JP401"  Part="1"
 AR Path="/57A0221A/579F6D99" Ref="JP501"  Part="1"
-F 0 "JP301" H 4640 3820 50  0000 C CNN
+F 0 "JP501" H 4640 3820 50  0000 C CNN
 F 1 "Jumper_NC_Small" H 4650 3680 50  0001 C CNN
-F 2 "" H 4640 3740 50  0001 C CNN
+F 2 "stmps:MADW__SMD-solder-bridge-narrow" H 4640 3740 50  0001 C CNN
 F 3 "" H 4640 3740 50  0000 C CNN
 	1    4640 3740
@@
 AR Path="/57A011F0/579F823F" Ref="R402"  Part="1"
 AR Path="/57A0221A/579F823F" Ref="R502"  Part="1"
-F 0 "R302" V 4600 3890 50  0000 L CNN
+F 0 "R502" V 4600 3890 50  0000 L CNN
 F 1 "100k" V 4730 3850 50  0000 L CNN
 F 2 "Resistors_SMD:R_0805_HandSoldering" H 4660 3930 50  0001 C CNN
@@
 AR Path="/57A011F0/579F8AB7" Ref="R403"  Part="1"
 AR Path="/57A0221A/579F8AB7" Ref="R503"  Part="1"
-F 0 "R303" V 4780 3230 50  0000 L CNN
+F 0 "R503" V 4780 3230 50  0000 L CNN
 F 1 "100k" V 4910 3190 50  0000 L CNN
 F 2 "Resistors_SMD:R_0805_HandSoldering" H 4840 3270 50  0001 C CNN
@@
 AR Path="/57A011F0/579FAB17" Ref="RV401"  Part="1"
 AR Path="/57A0221A/579FAB17" Ref="RV501"  Part="1"
-F 0 "RV301" H 4460 4000 50  0000 C CNN
+F 0 "RV501" H 4460 4000 50  0000 C CNN
 F 1 "100k" H 4460 4080 50  0000 C CNN
-F 2 "" H 4460 4080 50  0001 C CNN
+F 2 "stmps:BOURNS-TC33X-2" H 4460 4080 50  0001 C CNN
 F 3 "" H 4460 4080 50  0000 C CNN
 	1    4460 4080
@@
 AR Path="/57A011F0/579FAC77" Ref="R401"  Part="1"
 AR Path="/57A0221A/579FAC77" Ref="R501"  Part="1"
-F 0 "R301" H 4490 3850 50  0000 L CNN
+F 0 "R501" H 4490 3850 50  0000 L CNN
 F 1 "20k" H 4490 3790 50  0000 L CNN
 F 2 "Resistors_SMD:R_0805_HandSoldering" H 4460 3830 50  0001 C CNN

Commit message: Fix jumper names for steppers. Start prepping for layout.
Parts:
- JP201: value Jumper_NC_Small -> MS3
- JP202: value Jumper_NC_Small -> MS2
- JP203: value Jumper_NC_Small -> MS1
Changed lines of the file:
@@
 $Descr A4 11693 8268
 encoding utf-8
-Sheet 2 8
+Sheet 3 8
 Title ""
 Date ""
@@
 AR Path="/57A011F0/579F4813" Ref="U401"  Part="1"
 AR Path="/57A0221A/579F4813" Ref="U501"  Part="1"
-F 0 "U501" H 5890 2850 60  0000 C CNN
+F 0 "U301" H 5890 2850 60  0000 C CNN
 F 1 "A5984" H 5630 3670 60  0000 C CNN
 F 2 "stmps:TSSOP-24_4.4x7.8mm_Pitch0.65mm" H 5630 3670 60  0001 C CNN
@@
 AR Path="/57A011F0/579F48E9" Ref="C401"  Part="1"
 AR Path="/57A0221A/579F48E9" Ref="C501"  Part="1"
-F 0 "C501" H 5530 2790 50  0000 L CNN
+F 0 "C301" H 5530 2790 50  0000 L CNN
 F 1 "0.1uf" H 5530 2640 50  0000 L CNN
 F 2 "Capacitors_SMD:C_0805_HandSoldering" H 5520 2720 50  0001 C CNN
@@
 AR Path="/57A011F0/579F4A31" Ref="C402"  Part="1"
 AR Path="/57A0221A/579F4A31" Ref="C502"  Part="1"
-F 0 "C502" H 5990 2960 50  0000 L CNN
+F 0 "C302" H 5990 2960 50  0000 L CNN
 F 1 "0.1uf" H 5990 2810 50  0000 L CNN
 F 2 "Capacitors_SMD:C_0805_HandSoldering" H 5980 2890 50  0001 C CNN
@@
 AR Path="/57A011F0/579F5380" Ref="#PWR026"  Part="1"
 AR Path="/57A0221A/579F5380" Ref="#PWR028"  Part="1"
-F 0 "#PWR028" H 6530 2940 50  0001 C CNN
+F 0 "#PWR024" H 6530 2940 50  0001 C CNN
 F 1 "GND" H 6530 3040 50  0000 C CNN
 F 2 "" H 6530 3190 50  0000 C CNN
@@
 AR Path="/57A011F0/579F53B1" Ref="C403"  Part="1"
 AR Path="/57A0221A/579F53B1" Ref="C503"  Part="1"
-F 0 "C503" H 6540 3140 50  0000 L CNN
+F 0 "C303" H 6540 3140 50  0000 L CNN
 F 1 "100uf" H 6540 2990 50  0000 L CNN
 F 2 "Capacitors_SMD:c_elec_6.3x5.8" H 6530 3070 50  0001 C CNN
@@
 AR Path="/57A011F0/579F5CC2" Ref="R404"  Part="1"
 AR Path="/57A0221A/579F5CC2" Ref="R504"  Part="1"
-F 0 "R504" H 6440 4290 50  0000 L CNN
+F 0 "R304" H 6440 4290 50  0000 L CNN
 F 1 "0.05" H 6440 4230 50  0000 L CNN
 F 2 "Resistors_SMD:R_0805_HandSoldering" H 6410 4270 50  0001 C CNN
@@
 AR Path="/57A011F0/579F5D70" Ref="R405"  Part="1"
 AR Path="/57A0221A/579F5D70" Ref="R505"  Part="1"
-F 0 "R505" H 6700 4290 50  0000 L CNN
+F 0 "R305" H 6700 4290 50  0000 L CNN
 F 1 "0.05" H 6700 4230 50  0000 L CNN
 F 2 "Resistors_SMD:R_0805_HandSoldering" H 6670 4270 50  0001 C CNN
@@
 AR Path="/57A011F0/579F5F9F" Ref="#PWR027"  Part="1"
 AR Path="/57A0221A/579F5F9F" Ref="#PWR029"  Part="1"
-F 0 "#PWR029" H 6100 4460 50  0001 C CNN
+F 0 "#PWR025" H 6100 4460 50  0001 C CNN
 F 1 "GND" H 6100 4560 50  0000 C CNN
 F 2 "" H 6100 4710 50  0000 C CNN
@@
 AR Path="/57A011F0/579F6126" Ref="P401"  Part="1"
 AR Path="/57A0221A/579F6126" Ref="P501"  Part="1"
-F 0 "P501" H 6530 3950 50  0000 C CNN
+F 0 "P301" H 6530 3950 50  0000 C CNN
 F 1 "MOT" V 6630 3700 50  0000 C CNN
 F 2 "Pin_Headers:Pin_Header_Straight_1x04" H 6530 3700 50  0001 C CNN
@@
 AR Path="/57A011F0/579F6BCE" Ref="JP403"  Part="1"
 AR Path="/57A0221A/579F6BCE" Ref="JP503"  Part="1"
-F 0 "JP503" H 4990 3640 50  0000 C CNN
-F 1 "Jumper_NC_Small" H 5000 3500 50  0001 C CNN
+F 0 "JP303" H 4990 3640 50  0000 C CNN
+F 1 "MS1" H 5000 3500 50  0001 C CNN
 F 2 "stmps:MADW__SMD-solder-bridge-narrow" H 4990 3560 50  0001 C CNN
 F 3 "" H 4990 3560 50  0000 C CNN
@@
 AR Path="/57A011F0/579F6D26" Ref="JP402"  Part="1"
 AR Path="/57A0221A/579F6D26" Ref="JP502"  Part="1"
-F 0 "JP502" H 4810 3730 50  0000 C CNN
-F 1 "Jumper_NC_Small" H 4820 3590 50  0001 C CNN
+F 0 "JP302" H 4810 3730 50  0000 C CNN
+F 1 "MS2" H 4820 3590 50  0001 C CNN
 F 2 "stmps:MADW__SMD-solder-bridge-narrow" H 4810 3650 50  0001 C CNN
 F 3 "" H 4810 3650 50  0000 C CNN
@@
 AR Path="/57A011F0/579F6D99" Ref="JP401"  Part="1"
 AR Path="/57A0221A/579F6D99" Ref="JP501"  Part="1"
-F 0 "JP501" H 4640 3820 50  0000 C CNN
-F 1 "Jumper_NC_Small" H 4650 3680 50  0001 C CNN
+F 0 "JP301" H 4640 3820 50  0000 C CNN
+F 1 "MS3" H 4650 3680 50  0001 C CNN
 F 2 "stmps:MADW__SMD-solder-bridge-narrow" H 4640 3740 50  0001 C CNN
 F 3 "" H 4640 3740 50  0000 C CNN
@@
 AR Path="/57A011F0/579F823F" Ref="R402"  Part="1"
 AR Path="/57A0221A/579F823F" Ref="R502"  Part="1"
-F 0 "R502" V 4600 3890 50  0000 L CNN
+F 0 "R302" V 4600 3890 50  0000 L CNN
 F 1 "100k" V 4730 3850 50  0000 L CNN
 F 2 "Resistors_SMD:R_0805_HandSoldering" H 4660 3930 50  0001 C CNN
@@
 AR Path="/57A011F0/579F8AB7" Ref="R403"  Part="1"
 AR Path="/57A0221A/579F8AB7" Ref="R503"  Part="1"
-F 0 "R503" V 4780 3230 50  0000 L CNN
+F 0 "R303" V 4780 3230 50  0000 L CNN
 F 1 "100k" V 4910 3190 50  0000 L CNN
 F 2 "Resistors_SMD:R_0805_HandSoldering" H 4840 3270 50  0001 C CNN
@@
 AR Path="/57A011F0/579FAB17" Ref="RV401"  Part="1"
 AR Path="/57A0221A/579FAB17" Ref="RV501"  Part="1"
-F 0 "RV501" H 4460 4000 50  0000 C CNN
+F 0 "RV301" H 4460 4000 50  0000 C CNN
 F 1 "100k" H 4460 4080 50  0000 C CNN
 F 2 "stmps:BOURNS-TC33X-2" H 4460 4080 50  0001 C CNN
@@
 AR Path="/57A011F0/579FAC77" Ref="R401"  Part="1"
 AR Path="/57A0221A/579FAC77" Ref="R501"  Part="1"
-F 0 "R501" H 4490 3850 50  0000 L CNN
+F 0 "R301" H 4490 3850 50  0000 L CNN
 F 1 "20k" H 4490 3790 50  0000 L CNN
 F 2 "Resistors_SMD:R_0805_HandSoldering" H 4460 3830 50  0001 C CNN
