File: a5984_stepper.sch (KiCad schematic (older format))
At the start: 14 parts, among them P201 MOT, U201 A5984

Commit message: Complete routing, first pass.
Parts:
- added C404: 0.1uf, Capacitors_SMD:C_0805_HandSoldering, symbol C_Small
Connections:
- wire segments 43 -> 49
Changed lines of the file:
@@
 $Descr A4 11693 8268
 encoding utf-8
-Sheet 3 8
+Sheet 4 8
 Title ""
 Date ""
@@
 AR Path="/57A011F0/579F4813" Ref="U401"  Part="1"
 AR Path="/57A0221A/579F4813" Ref="U501"  Part="1"
-F 0 "U301" H 5890 2850 60  0000 C CNN
+F 0 "U401" H 5890 2850 60  0000 C CNN
 F 1 "A5984" H 5630 3670 60  0000 C CNN
 F 2 "stmps:TSSOP-24_4.4x7.8mm_Pitch0.65mm" H 5630 3670 60  0001 C CNN
@@
 AR Path="/57A011F0/579F48E9" Ref="C401"  Part="1"
 AR Path="/57A0221A/579F48E9" Ref="C501"  Part="1"
-F 0 "C301" H 5530 2790 50  0000 L CNN
+F 0 "C401" H 5530 2790 50  0000 L CNN
 F 1 "0.1uf" H 5530 2640 50  0000 L CNN
 F 2 "Capacitors_SMD:C_0805_HandSoldering" H 5520 2720 50  0001 C CNN
@@
 AR Path="/57A011F0/579F4A31" Ref="C402"  Part="1"
 AR Path="/57A0221A/579F4A31" Ref="C502"  Part="1"
-F 0 "C302" H 5990 2960 50  0000 L CNN
+F 0 "C402" H 5990 2960 50  0000 L CNN
 F 1 "0.1uf" H 5990 2810 50  0000 L CNN
 F 2 "Capacitors_SMD:C_0805_HandSoldering" H 5980 2890 50  0001 C CNN
@@
 +12v
 $Comp
-L GND #PWR022
+L GND #PWR020
 U 1 1 579F5380
-P 6530 3190
-AR Path="/579F3F70/579F5380" Ref="#PWR022"  Part="1"
-AR Path="/57A00526/579F5380" Ref="#PWR024"  Part="1"
-AR Path="/57A011F0/579F5380" Ref="#PWR026"  Part="1"
-AR Path="/57A0221A/579F5380" Ref="#PWR028"  Part="1"
-F 0 "#PWR024" H 6530 2940 50  0001 C CNN
-F 1 "GND" H 6530 3040 50  0000 C CNN
-F 2 "" H 6530 3190 50  0000 C CNN
-F 3 "" H 6530 3190 50  0000 C CNN
-	1    6530 3190
+P 6430 3220
+AR Path="/579F3F70/579F5380" Ref="#PWR020"  Part="1"
+AR Path="/57A00526/579F5380" Ref="#PWR022"  Part="1"
+AR Path="/57A011F0/579F5380" Ref="#PWR024"  Part="1"
+AR Path="/57A0221A/579F5380" Ref="#PWR026"  Part="1"
+F 0 "#PWR024" H 6430 2970 50  0001 C CNN
+F 1 "GND" H 6430 3070 50  0000 C CNN
+F 2 "" H 6430 3220 50  0000 C CNN
+F 3 "" H 6430 3220 50  0000 C CNN
+	1    6430 3220
 	1    0    0    -1
 $EndComp
@@
 AR Path="/57A011F0/579F53B1" Ref="C403"  Part="1"
 AR Path="/57A0221A/579F53B1" Ref="C503"  Part="1"
-F 0 "C303" H 6540 3140 50  0000 L CNN
+F 0 "C403" H 6540 3140 50  0000 L CNN
 F 1 "100uf" H 6540 2990 50  0000 L CNN
 F 2 "Capacitors_SMD:c_elec_6.3x5.8" H 6530 3070 50  0001 C CNN
@@
 AR Path="/57A011F0/579F5CC2" Ref="R404"  Part="1"
 AR Path="/57A0221A/579F5CC2" Ref="R504"  Part="1"
-F 0 "R304" H 6440 4290 50  0000 L CNN
+F 0 "R404" H 6440 4290 50  0000 L CNN
 F 1 "0.05" H 6440 4230 50  0000 L CNN
 F 2 "Resistors_SMD:R_0805_HandSoldering" H 6410 4270 50  0001 C CNN
@@
 AR Path="/57A011F0/579F5D70" Ref="R405"  Part="1"
 AR Path="/57A0221A/579F5D70" Ref="R505"  Part="1"
-F 0 "R305" H 6700 4290 50  0000 L CNN
+F 0 "R405" H 6700 4290 50  0000 L CNN
 F 1 "0.05" H 6700 4230 50  0000 L CNN
 F 2 "Resistors_SMD:R_0805_HandSoldering" H 6670 4270 50  0001 C CNN
@@
 $EndComp
 $Comp
-L GND #PWR023
+L GND #PWR021
 U 1 1 579F5F9F
 P 6100 4710
-AR Path="/579F3F70/579F5F9F" Ref="#PWR023"  Part="1"
-AR Path="/57A00526/579F5F9F" Ref="#PWR025"  Part="1"
-AR Path="/57A011F0/579F5F9F" Ref="#PWR027"  Part="1"
-AR Path="/57A0221A/579F5F9F" Ref="#PWR029"  Part="1"
+AR Path="/579F3F70/579F5F9F" Ref="#PWR021"  Part="1"
+AR Path="/57A00526/579F5F9F" Ref="#PWR023"  Part="1"
+AR Path="/57A011F0/579F5F9F" Ref="#PWR025"  Part="1"
+AR Path="/57A0221A/579F5F9F" Ref="#PWR027"  Part="1"
 F 0 "#PWR025" H 6100 4460 50  0001 C CNN
 F 1 "GND" H 6100 4560 50  0000 C CNN
@@
 F 3 "" H 6100 4710 50  0000 C CNN
 	1    6100 4710
-	1    0    0    -1
-$EndComp
-$Comp
-L CONN_01X04 P201
-U 1 1 579F6126
-P 6530 3700
-AR Path="/579F3F70/579F6126" Ref="P201"  Part="1"
-AR Path="/57A00526/579F6126" Ref="P301"  Part="1"
-AR Path="/57A011F0/579F6126" Ref="P401"  Part="1"
-AR Path="/57A0221A/579F6126" Ref="P501"  Part="1"
-F 0 "P301" H 6530 3950 50  0000 C CNN
-F 1 "MOT" V 6630 3700 50  0000 C CNN
-F 2 "Pin_Headers:Pin_Header_Straight_1x04" H 6530 3700 50  0001 C CNN
-F 3 "" H 6530 3700 50  0000 C CNN
-	1    6530 3700
 	1    0    0    -1
 $EndComp
@@
 AR Path="/57A011F0/579F6BCE" Ref="JP403"  Part="1"
 AR Path="/57A0221A/579F6BCE" Ref="JP503"  Part="1"
-F 0 "JP303" H 4990 3640 50  0000 C CNN
+F 0 "JP403" H 4990 3640 50  0000 C CNN
 F 1 "MS1" H 5000 3500 50  0001 C CNN
 F 2 "stmps:MADW__SMD-solder-bridge-narrow" H 4990 3560 50  0001 C CNN
@@
 AR Path="/57A011F0/579F6D26" Ref="JP402"  Part="1"
 AR Path="/57A0221A/579F6D26" Ref="JP502"  Part="1"
-F 0 "JP302" H 4810 3730 50  0000 C CNN
+F 0 "JP402" H 4810 3730 50  0000 C CNN
 F 1 "MS2" H 4820 3590 50  0001 C CNN
 F 2 "stmps:MADW__SMD-solder-bridge-narrow" H 4810 3650 50  0001 C CNN
@@
 AR Path="/57A011F0/579F6D99" Ref="JP401"  Part="1"
 AR Path="/57A0221A/579F6D99" Ref="JP501"  Part="1"
-F 0 "JP301" H 4640 3820 50  0000 C CNN
+F 0 "JP401" H 4640 3820 50  0000 C CNN
 F 1 "MS3" H 4650 3680 50  0001 C CNN
 F 2 "stmps:MADW__SMD-solder-bridge-narrow" H 4640 3740 50  0001 C CNN
@@
 AR Path="/57A011F0/579F823F" Ref="R402"  Part="1"
 AR Path="/57A0221A/579F823F" Ref="R502"  Part="1"
-F 0 "R302" V 4600 3890 50  0000 L CNN
+F 0 "R402" V 4600 3890 50  0000 L CNN
 F 1 "100k" V 4730 3850 50  0000 L CNN
 F 2 "Resistors_SMD:R_0805_HandSoldering" H 4660 3930 50  0001 C CNN
@@
 AR Path="/57A011F0/579F8AB7" Ref="R403"  Part="1"
 AR Path="/57A0221A/579F8AB7" Ref="R503"  Part="1"
-F 0 "R303" V 4780 3230 50  0000 L CNN
+F 0 "R403" V 4780 3230 50  0000 L CNN
 F 1 "100k" V 4910 3190 50  0000 L CNN
 F 2 "Resistors_SMD:R_0805_HandSoldering" H 4840 3270 50  0001 C CNN
@@
 AR Path="/57A011F0/579FAB17" Ref="RV401"  Part="1"
 AR Path="/57A0221A/579FAB17" Ref="RV501"  Part="1"
-F 0 "RV301" H 4460 4000 50  0000 C CNN
+F 0 "RV401" H 4460 4000 50  0000 C CNN
 F 1 "100k" H 4460 4080 50  0000 C CNN
 F 2 "stmps:BOURNS-TC33X-2" H 4460 4080 50  0001 C CNN
@@
 AR Path="/57A011F0/579FAC77" Ref="R401"  Part="1"
 AR Path="/57A0221A/579FAC77" Ref="R501"  Part="1"
-F 0 "R301" H 4490 3850 50  0000 L CNN
+F 0 "R401" H 4490 3850 50  0000 L CNN
 F 1 "20k" H 4490 3790 50  0000 L CNN
 F 2 "Resistors_SMD:R_0805_HandSoldering" H 4460 3830 50  0001 C CNN
@@
 Connection ~ 6530 2890
 Wire Wire Line
-	6530 3170 6530 3190
+	6530 3220 6530 3170
 Wire Wire Line
 	5580 4530 5580 4660
@@
 	6670 4040 6110 4040
 Wire Wire Line
-	6110 3480 6330 3480
-Wire Wire Line
-	6330 3480 6330 3550
-Wire Wire Line
-	6330 3650 6110 3650
-Wire Wire Line
-	6110 3650 6110 3570
-Wire Wire Line
 	6110 3750 6330 3750
 Wire Wire Line
@@
 	4460 4230 4460 4660
 Connection ~ 5580 4660
+$Comp
+L CONN_01X04 P201
+U 1 1 579F6126
+P 6530 3700
+AR Path="/579F3F70/579F6126" Ref="P201"  Part="1"
+AR Path="/57A00526/579F6126" Ref="P301"  Part="1"
+AR Path="/57A011F0/579F6126" Ref="P401"  Part="1"
+AR Path="/57A0221A/579F6126" Ref="P501"  Part="1"
+F 0 "P401" H 6530 3950 50  0000 C CNN
+F 1 "MOT" V 6630 3700 50  0000 C CNN
+F 2 "Pin_Headers:Pin_Header_Straight_1x04" H 6530 3700 50  0001 C CNN
+F 3 "" H 6530 3700 50  0000 C CNN
+	1    6530 3700
+	1    0    0    -1
+$EndComp
+Wire Wire Line
+	6110 3570 6220 3570
+Wire Wire Line
+	6220 3570 6220 3550
+Wire Wire Line
+	6220 3550 6330 3550
+Wire Wire Line
+	6330 3650 6250 3650
+Wire Wire Line
+	6250 3650 6250 3480
+Wire Wire Line
+	6250 3480 6110 3480
+$Comp
+L C_Small C404
+U 1 1 57A1ADDF
+P 6330 3070
+AR Path="/57A011F0/57A1ADDF" Ref="C404"  Part="1"
+AR Path="/579F3F70/57A1ADDF" Ref="C204"  Part="1"
+AR Path="/57A00526/57A1ADDF" Ref="C304"  Part="1"
+AR Path="/57A0221A/57A1ADDF" Ref="C504"  Part="1"
+F 0 "C404" H 6340 3140 50  0000 L CNN
+F 1 "0.1uf" H 6340 2990 50  0000 L CNN
+F 2 "Capacitors_SMD:C_0805_HandSoldering" H 6330 3070 50  0001 C CNN
+F 3 "" H 6330 3070 50  0000 C CNN
+	1    6330 3070
+	1    0    0    -1
+$EndComp
+Wire Wire Line
+	6330 2970 6330 2890
+Connection ~ 6330 2890
+Wire Wire Line
+	6330 3170 6330 3220
+Wire Wire Line
+	6330 3220 6530 3220
+Connection ~ 6430 3220
+Wire Wire Line
+	5500 4530 5500 4660
+Connection ~ 5500 4660
 $EndSCHEMATC

Commit message: Corrected resistors and rail for vREF.
Parts:
- R201: value 20k -> 200k
- R204, R205: value 0.05 -> 0.1
- RV201: MPN (none) -> TC33X-2-104E
- U201: MPN (none) -> A5984GLPTR-T
Connections:
- wire segments 49 -> 50
Changed lines of the file:
@@
 $Descr A4 11693 8268
 encoding utf-8
-Sheet 4 8
+Sheet 2 8
 Title ""
 Date ""
@@
 AR Path="/57A011F0/579F4813" Ref="U401"  Part="1"
 AR Path="/57A0221A/579F4813" Ref="U501"  Part="1"
-F 0 "U401" H 5890 2850 60  0000 C CNN
+F 0 "U201" H 5890 2850 60  0000 C CNN
 F 1 "A5984" H 5630 3670 60  0000 C CNN
 F 2 "stmps:TSSOP-24_4.4x7.8mm_Pitch0.65mm" H 5630 3670 60  0001 C CNN
 F 3 "" H 5630 3670 60  0000 C CNN
+F 4 "A5984GLPTR-T" H 5630 3670 60  0001 C CNN "MPN"
 	1    5630 3670
 	1    0    0    -1
@@
 AR Path="/57A011F0/579F48E9" Ref="C401"  Part="1"
 AR Path="/57A0221A/579F48E9" Ref="C501"  Part="1"
-F 0 "C401" H 5530 2790 50  0000 L CNN
+F 0 "C201" H 5530 2790 50  0000 L CNN
 F 1 "0.1uf" H 5530 2640 50  0000 L CNN
 F 2 "Capacitors_SMD:C_0805_HandSoldering" H 5520 2720 50  0001 C CNN
@@
 AR Path="/57A011F0/579F4A31" Ref="C402"  Part="1"
 AR Path="/57A0221A/579F4A31" Ref="C502"  Part="1"
-F 0 "C402" H 5990 2960 50  0000 L CNN
+F 0 "C202" H 5990 2960 50  0000 L CNN
 F 1 "0.1uf" H 5990 2810 50  0000 L CNN
 F 2 "Capacitors_SMD:C_0805_HandSoldering" H 5980 2890 50  0001 C CNN
@@
 AR Path="/57A011F0/579F5380" Ref="#PWR024"  Part="1"
 AR Path="/57A0221A/579F5380" Ref="#PWR026"  Part="1"
-F 0 "#PWR024" H 6430 2970 50  0001 C CNN
+F 0 "#PWR020" H 6430 2970 50  0001 C CNN
 F 1 "GND" H 6430 3070 50  0000 C CNN
 F 2 "" H 6430 3220 50  0000 C CNN
@@
 AR Path="/57A011F0/579F53B1" Ref="C403"  Part="1"
 AR Path="/57A0221A/579F53B1" Ref="C503"  Part="1"
-F 0 "C403" H 6540 3140 50  0000 L CNN
+F 0 "C203" H 6540 3140 50  0000 L CNN
 F 1 "100uf" H 6540 2990 50  0000 L CNN
 F 2 "Capacitors_SMD:c_elec_6.3x5.8" H 6530 3070 50  0001 C CNN
@@
 AR Path="/57A011F0/579F5CC2" Ref="R404"  Part="1"
 AR Path="/57A0221A/579F5CC2" Ref="R504"  Part="1"
-F 0 "R404" H 6440 4290 50  0000 L CNN
-F 1 "0.05" H 6440 4230 50  0000 L CNN
+F 0 "R204" H 6440 4290 50  0000 L CNN
+F 1 "0.1" H 6440 4230 50  0000 L CNN
 F 2 "Resistors_SMD:R_0805_HandSoldering" H 6410 4270 50  0001 C CNN
 F 3 "" H 6410 4270 50  0000 C CNN
@@
 AR Path="/57A011F0/579F5D70" Ref="R405"  Part="1"
 AR Path="/57A0221A/579F5D70" Ref="R505"  Part="1"
-F 0 "R405" H 6700 4290 50  0000 L CNN
-F 1 "0.05" H 6700 4230 50  0000 L CNN
+F 0 "R205" H 6700 4290 50  0000 L CNN
+F 1 "0.1" H 6700 4230 50  0000 L CNN
 F 2 "Resistors_SMD:R_0805_HandSoldering" H 6670 4270 50  0001 C CNN
 F 3 "" H 6670 4270 50  0000 C CNN
@@
 AR Path="/57A011F0/579F5F9F" Ref="#PWR025"  Part="1"
 AR Path="/57A0221A/579F5F9F" Ref="#PWR027"  Part="1"
-F 0 "#PWR025" H 6100 4460 50  0001 C CNN
+F 0 "#PWR021" H 6100 4460 50  0001 C CNN
 F 1 "GND" H 6100 4560 50  0000 C CNN
 F 2 "" H 6100 4710 50  0000 C CNN
@@
 AR Path="/57A011F0/579F6BCE" Ref="JP403"  Part="1"
 AR Path="/57A0221A/579F6BCE" Ref="JP503"  Part="1"
-F 0 "JP403" H 4990 3640 50  0000 C CNN
+F 0 "JP203" H 4990 3640 50  0000 C CNN
 F 1 "MS1" H 5000 3500 50  0001 C CNN
 F 2 "stmps:MADW__SMD-solder-bridge-narrow" H 4990 3560 50  0001 C CNN
@@
 AR Path="/57A011F0/579F6D26" Ref="JP402"  Part="1"
 AR Path="/57A0221A/579F6D26" Ref="JP502"  Part="1"
-F 0 "JP402" H 4810 3730 50  0000 C CNN
+F 0 "JP202" H 4810 3730 50  0000 C CNN
 F 1 "MS2" H 4820 3590 50  0001 C CNN
 F 2 "stmps:MADW__SMD-solder-bridge-narrow" H 4810 3650 50  0001 C CNN
@@
 AR Path="/57A011F0/579F6D99" Ref="JP401"  Part="1"
 AR Path="/57A0221A/579F6D99" Ref="JP501"  Part="1"
-F 0 "JP401" H 4640 3820 50  0000 C CNN
+F 0 "JP201" H 4640 3820 50  0000 C CNN
 F 1 "MS3" H 4650 3680 50  0001 C CNN
 F 2 "stmps:MADW__SMD-solder-bridge-narrow" H 4640 3740 50  0001 C CNN
@@
 	1    0    0    -1
 $EndComp
-Text GLabel 4410 3560 0    60   Input ~ 0
+Text GLabel 4540 3360 0    60   Input ~ 0
 +3.3v
 $Comp
@@
 AR Path="/57A011F0/579F823F" Ref="R402"  Part="1"
 AR Path="/57A0221A/579F823F" Ref="R502"  Part="1"
-F 0 "R402" V 4600 3890 50  0000 L CNN
+F 0 "R202" V 4600 3890 50  0000 L CNN
 F 1 "100k" V 4730 3850 50  0000 L CNN
 F 2 "Resistors_SMD:R_0805_HandSoldering" H 4660 3930 50  0001 C CNN
@@
 AR Path="/57A011F0/579F8AB7" Ref="R403"  Part="1"
 AR Path="/57A0221A/579F8AB7" Ref="R503"  Part="1"
-F 0 "R403" V 4780 3230 50  0000 L CNN
+F 0 "R203" V 4780 3230 50  0000 L CNN
 F 1 "100k" V 4910 3190 50  0000 L CNN
 F 2 "Resistors_SMD:R_0805_HandSoldering" H 4840 3270 50  0001 C CNN
@@
 AR Path="/57A011F0/579FAB17" Ref="RV401"  Part="1"
 AR Path="/57A0221A/579FAB17" Ref="RV501"  Part="1"
-F 0 "RV401" H 4460 4000 50  0000 C CNN
+F 0 "RV201" H 4460 4000 50  0000 C CNN
 F 1 "100k" H 4460 4080 50  0000 C CNN
 F 2 "stmps:BOURNS-TC33X-2" H 4460 4080 50  0001 C CNN
 F 3 "" H 4460 4080 50  0000 C CNN
+F 4 "TC33X-2-104E" H 4460 4080 60  0001 C CNN "MPN"
 	1    4460 4080
 	0    1    1    0
@@
 AR Path="/57A011F0/579FAC77" Ref="R401"  Part="1"
 AR Path="/57A0221A/579FAC77" Ref="R501"  Part="1"
-F 0 "R401" H 4490 3850 50  0000 L CNN
-F 1 "20k" H 4490 3790 50  0000 L CNN
+F 0 "R201" H 4490 3850 50  0000 L CNN
+F 1 "200k" H 4490 3790 50  0000 L CNN
 F 2 "Resistors_SMD:R_0805_HandSoldering" H 4460 3830 50  0001 C CNN
 F 3 "" H 4460 3830 50  0000 C CNN
@@
 Wire Wire Line
 	4540 3270 4540 3930
-Wire Wire Line
-	4410 3560 4890 3560
 Connection ~ 4540 3560
 Wire Wire Line
@@
 Wire Wire Line
 	4610 4080 5130 4080
-Wire Wire Line
-	4460 3730 4460 3560
-Connection ~ 4460 3560
 Wire Wire Line
 	4460 4230 4460 4660
@@
 AR Path="/57A011F0/579F6126" Ref="P401"  Part="1"
 AR Path="/57A0221A/579F6126" Ref="P501"  Part="1"
-F 0 "P401" H 6530 3950 50  0000 C CNN
+F 0 "P201" H 6530 3950 50  0000 C CNN
 F 1 "MOT" V 6630 3700 50  0000 C CNN
 F 2 "Pin_Headers:Pin_Header_Straight_1x04" H 6530 3700 50  0001 C CNN
@@
 AR Path="/57A00526/57A1ADDF" Ref="C304"  Part="1"
 AR Path="/57A0221A/57A1ADDF" Ref="C504"  Part="1"
-F 0 "C404" H 6340 3140 50  0000 L CNN
+F 0 "C204" H 6340 3140 50  0000 L CNN
 F 1 "0.1uf" H 6340 2990 50  0000 L CNN
 F 2 "Capacitors_SMD:C_0805_HandSoldering" H 6330 3070 50  0001 C CNN
@@
 	5500 4530 5500 4660
 Connection ~ 5500 4660
+Text GLabel 4410 3680 0    60   Input ~ 0
++12v
+Wire Wire Line
+	4540 3560 4890 3560
+Wire Wire Line
+	4460 3730 4460 3680
+Wire Wire Line
+	4460 3680 4410 3680
 $EndSCHEMATC

Commit message: Fix USB connection. Cleanups.
Changed lines of the file:
@@
 +12v
 $Comp
-L GND #PWR020
+L GND #PWR021
 U 1 1 579F5380
-P 6430 3220
-AR Path="/579F3F70/579F5380" Ref="#PWR020"  Part="1"
-AR Path="/57A00526/579F5380" Ref="#PWR022"  Part="1"
-AR Path="/57A011F0/579F5380" Ref="#PWR024"  Part="1"
-AR Path="/57A0221A/579F5380" Ref="#PWR026"  Part="1"
-F 0 "#PWR020" H 6430 2970 50  0001 C CNN
-F 1 "GND" H 6430 3070 50  0000 C CNN
-F 2 "" H 6430 3220 50  0000 C CNN
-F 3 "" H 6430 3220 50  0000 C CNN
-	1    6430 3220
+P 6460 3220
+AR Path="/579F3F70/579F5380" Ref="#PWR021"  Part="1"
+AR Path="/57A00526/579F5380" Ref="#PWR023"  Part="1"
+AR Path="/57A011F0/579F5380" Ref="#PWR025"  Part="1"
+AR Path="/57A0221A/579F5380" Ref="#PWR027"  Part="1"
+F 0 "#PWR027" H 6460 2970 50  0001 C CNN
+F 1 "GND" H 6460 3070 50  0000 C CNN
+F 2 "" H 6460 3220 50  0000 C CNN
+F 3 "" H 6460 3220 50  0000 C CNN
+	1    6460 3220
 	1    0    0    -1
 $EndComp
@@
 L CP1_Small C203
 U 1 1 579F53B1
-P 6530 3070
+P 6590 3070
 AR Path="/579F3F70/579F53B1" Ref="C203"  Part="1"
 AR Path="/57A00526/579F53B1" Ref="C303"  Part="1"
 AR Path="/57A011F0/579F53B1" Ref="C403"  Part="1"
 AR Path="/57A0221A/579F53B1" Ref="C503"  Part="1"
-F 0 "C203" H 6540 3140 50  0000 L CNN
-F 1 "100uf" H 6540 2990 50  0000 L CNN
-F 2 "Capacitors_SMD:c_elec_6.3x5.8" H 6530 3070 50  0001 C CNN
-F 3 "" H 6530 3070 50  0000 C CNN
-F 4 "UWT1V101MCL1GS" H 6530 3070 60  0001 C CNN "MPN"
-	1    6530 3070
+F 0 "C203" H 6600 3140 50  0000 L CNN
+F 1 "100uf" H 6600 2990 50  0000 L CNN
+F 2 "Capacitors_SMD:c_elec_6.3x5.8" H 6590 3070 50  0001 C CNN
+F 3 "" H 6590 3070 50  0000 C CNN
+F 4 "UWT1V101MCL1GS" H 6590 3070 60  0001 C CNN "MPN"
+	1    6590 3070
 	1    0    0    -1
 $EndComp
@@
 $EndComp
 $Comp
-L GND #PWR021
+L GND #PWR022
 U 1 1 579F5F9F
 P 6100 4710
-AR Path="/579F3F70/579F5F9F" Ref="#PWR021"  Part="1"
-AR Path="/57A00526/579F5F9F" Ref="#PWR023"  Part="1"
-AR Path="/57A011F0/579F5F9F" Ref="#PWR025"  Part="1"
-AR Path="/57A0221A/579F5F9F" Ref="#PWR027"  Part="1"
-F 0 "#PWR021" H 6100 4460 50  0001 C CNN
+AR Path="/579F3F70/579F5F9F" Ref="#PWR022"  Part="1"
+AR Path="/57A00526/579F5F9F" Ref="#PWR024"  Part="1"
+AR Path="/57A011F0/579F5F9F" Ref="#PWR026"  Part="1"
+AR Path="/57A0221A/579F5F9F" Ref="#PWR028"  Part="1"
+F 0 "#PWR028" H 6100 4460 50  0001 C CNN
 F 1 "GND" H 6100 4560 50  0000 C CNN
 F 2 "" H 6100 4710 50  0000 C CNN
@@
 Connection ~ 6230 2890
 Wire Wire Line
-	6530 2970 6530 2890
-Connection ~ 6530 2890
-Wire Wire Line
-	6530 3220 6530 3170
-Wire Wire Line
-	5580 4530 5580 4660
+	6590 2970 6590 2890
+Connection ~ 6590 2890
+Wire Wire Line
+	6590 3220 6590 3170
+Wire Wire Line
+	5580 4660 5580 4530
 Wire Wire Line
 	4460 4660 6670 4660
@@
 	6330 3170 6330 3220
 Wire Wire Line
-	6330 3220 6530 3220
-Connection ~ 6430 3220
+	6330 3220 6590 3220
+Connection ~ 6460 3220
 Wire Wire Line
 	5500 4530 5500 4660
