File: STMPS.kicad_pcb (KiCad board)
At the start: 2 copper layers, 85.9 x 56.9 mm, 116 parts, among them P101 12v IN, P102 12v, P103 USB_OTG, P104 E0_THERM, P105 X_STOP, P106 SWD, P107 BED_THERM, P108 Y_STOP, P109 Z_STOP, P201 MOT, P301 MOT, P401 MOT, P501 MOT, P601 LP_OUT, P701 OUT, P801 OUT, Q601 SSM3K333, Q701 IPP039N04L, Q801 IPP039N04L, U101 AOZ8904, U102 LM1117-3.3v, U103 STM32F411RCTx, U105 CHIP-TOP, U201 A5984, U301 A5984, U401 A5984, U501 A5984, Y101 Crystal

Commit message: Alpha 2 board layout.
Parts:
- added R107: 4.7k, Resistors_SMD:R_0805_HandSoldering, B.Cu at (123.7, 145.3)
- added REF**: Symbol_OSHW-Logo_SilkScreen, Symbols:Symbol_OSHW-Logo_SilkScreen, B.Cu at (101.3, 148.3)
- D101, D103, R101: moved to B.Cu
- P103: footprint Connect:USB_Micro-B -> stmps:USB_Micro-B-ebay
- moved P103 114.3 mm to (174.6, 149.4), turned to 90 degrees
- moved U101 110.3 mm to (169.9, 149.4), turned to 270 degrees
- moved U105 96.9 mm to (128.8, 132.8)
- moved P106 80.5 mm to (163.4, 148.5), turned to 270 degrees
- moved R104 78.2 mm to (143.3, 148.1)
- moved JP101 77.2 mm to (145.0, 151.9), turned to 180 degrees
- moved R101 56.3 mm to (114.0, 112.2), turned to 90 degrees
- moved P102 53.3 mm to (111.9, 111.0)
- moved D101 52.9 mm to (115.8, 112.3), turned to 270 degrees
- moved D103 37.6 mm to (147.9, 145.2), turned to 270 degrees
- moved D102 32.5 mm to (107.4, 148.8), turned to 90 degrees
- moved R102 32.4 mm to (109.7, 148.7)
- moved U102 23.0 mm to (151.9, 141.4), turned to 90 degrees
- moved P104 22.9 mm to (125.0, 152.4), turned to 270 degrees
- moved C102 22.1 mm to (145.8, 145.3), turned to 270 degrees
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Connections:
- net /SCL renamed Net-(U103-Pad58)
- net /SDA renamed Net-(U103-Pad59)
- U101 pad 3: /USB_DM -> /USB_DP
- U101 pad 4: /USB_DP -> /USB_DM
- U103 pad 10: /E0_Stepper/ENABLE -> /X_Stepper/ENABLE
- U103 pad 11: Net-(U103-Pad11) -> /CHIP_1_WIRE
- U103 pad 2: /X_Stepper/ENABLE -> /E0_Stepper/DIR
- U103 pad 23: Net-(U103-Pad23) -> /BED_FET/PWM_IN
- U103 pad 3: /X_Stepper/DIR -> /E0_Stepper/STEP
- U103 pad 4: /X_Stepper/STEP -> /E0_Stepper/ENABLE
- U103 pad 54: /BED_FET/PWM_IN -> Net-(U103-Pad54)
- U103 pad 62: /CHIP_1_WIRE -> Net-(U103-Pad62)
- U103 pad 8: /E0_Stepper/STEP -> /X_Stepper/DIR
- U103 pad 9: /E0_Stepper/DIR -> /X_Stepper/STEP
Routing:
- net +3.3v: track 39.9 -> 186.7 mm, vias 4 -> 13
- net GND: track 16.5 -> 92.3 mm, vias 3 -> 53
- net /USB_DP: track 0.00 -> 72.7 mm, vias 0 -> 2
- net /USB_DM: track 0.00 -> 72.6 mm, vias 0 -> 4
- net /E0_Stepper/DIR: track 0.00 -> 53.7 mm
- net /+5v: track 0.00 -> 50.2 mm, vias 0 -> 3
- net /SWCLK: track 0.00 -> 43.2 mm
- net /E0_Stepper/STEP: track 0.00 -> 42.7 mm
- net /USART1_TX: track 0.00 -> 42.4 mm, vias 0 -> 2
- net /E0_Stepper/ENABLE: track 0.00 -> 42.1 mm
- net /USART1_RX: track 0.00 -> 40.1 mm, vias 0 -> 2
- net /X_Stepper/DIR: track 0.00 -> 39.3 mm
- net /SWDIO: track 0.00 -> 33.9 mm, vias 0 -> 2
- net /BED_THERM: track 5.22 -> 37.1 mm
- net /X_Stepper/STEP: track 0.00 -> 28.4 mm
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- added copper zone on B.Cu, net GND
Other:
- board size 85.9 x 56.9 mm -> 85.9 x 44.7 mm
- board text added: "STMPS Alpha 2 8/2016"
- board text removed: "STMPS Rev. Alpha"
