File: STMPS.sch (KiCad schematic (older format))
At the start: 20 parts

Commit message: Possibly finished schematic.
Parts:
- removed C? (x5): 100nf, symbol C
- removed R?: R, symbol R
- added C101: 100uf, symbol CP_Small
- added C106, C108, C110, C111, C112: 100nf, symbol C_Small
- added C115: 0.1uf, symbol C_Small
- added C116, C117: 10uf, symbol C_Small
- added D101: 12v_PWR, symbol Led_Small
- added D102: 3v_PWR, symbol Led_Small
- added P102: 12v, symbol CONN_02X03
- added P103: USB_OTG, symbol USB_OTG
- added P104: E0_THERM, symbol CONN_01X02
- added P105: X_STOP, symbol CONN_01X03
- added P106: CONN_01X06, symbol CONN_01X06
- added P107: BED_THERM, symbol CONN_01X02
- added P108: Y_STOP, symbol CONN_01X03
- added P109: Z_STOP, symbol CONN_01X03
- added R101: 560, symbol R_Small
- added R102: 56, symbol R_Small
- added R104: 100k, symbol R_Small
- added R105, R106, R107, R108: 4.7k, symbol R_Small
- added SW101: RST, symbol SW_PUSH_SMALL
- added U101: PRTR5V0U4D, symbol PRTR5V0U4D
- added U104: M24C04, symbol 24C16
- added W101, W102, W103, W104: TEST_1P, symbol TEST_1P
- C102, C103, C104, C105, C107: renamed from C?; symbol C -> C_Small
- C109, C114: renamed from C?; symbol CP -> CP_Small
- C113: renamed from C?; symbol CP -> C_Small
- P101: renamed from P?; value CONN_02X02 -> 12v IN
- R103: renamed from R?; symbol R -> R_Small
- Y101: renamed from Y?; symbol Crystal -> Crystal_Small
- gave numbers to parts that had none: 3
Connections:
- net labels added: +12V, BED_PWM, BED_THERM, E0_DIR, E0_ENABLE, E0_PWM, E0_STEP, E0_THERM, FAN_PWM, NRST, SCL, SDA, SWCLK, SWDIO, SWO, USB_DN, USB_DP, X_DIR, X_ENABLE, X_STEP, X_STOP, Y_DIR, Y_ENABLE, Y_STEP, Y_STOP, Z_DIR, Z_ENABLE, Z_STEP, Z_STOP
- net labels removed: VDD
- wire segments 89 -> 163
- no-connect marks 0 -> 28

Commit message: Start working on footprint assignments.
Parts:
- C102, C103, C104, C105, C106, C107, C108, C110, C111, C112, C113, C115, C116, C117: footprint (none) -> Capacitors_SMD:C_0805_HandSoldering
- D101, D102: footprint (none) -> LEDs:LED_0805
- JP101: symbol JUMPER -> Jumper_NC_Small
- P104, P107: footprint (none) -> Pin_Headers:Pin_Header_Straight_1x02
- P105, P108, P109: footprint (none) -> Pin_Headers:Pin_Header_Straight_1x03
- P106: value CONN_01X06 -> SWD; footprint (none) -> Pin_Headers:Pin_Header_Straight_1x06
- R101, R102, R103, R104, R105, R106, R107, R108: footprint (none) -> Resistors_SMD:R_0805_HandSoldering
- U103: footprint LQFP64 -> (none)
- W101, W102, W103, W104: footprint (none) -> Connect:PINTST
Connections:
- wire segments 163 -> 118

Commit message: Finish assigning footprints.
Parts:
- added C118: 0.1uf, Capacitors_SMD:C_0805_HandSoldering, symbol C_Small
- C101: footprint (none) -> Capacitors_SMD:c_elec_6.3x5.8; MPN (none) -> 35TZV100M6.3X8
- C109, C114: footprint (none) -> Capacitors_SMD:C_0805_HandSoldering; symbol CP_Small -> C_Small
- JP101: footprint (none) -> stmps:MADW__SMD-solder-bridge-narrow
- P101: footprint (none) -> stmps:5EHDRC_1x04; symbol CONN_02X02 -> CONN_01X04
- P102: footprint (none) -> Pin_Headers:Pin_Header_Straight_2x03
- P103: footprint (none) -> Connect:USB_Micro-B
- SW101: footprint (none) -> Buttons_Switches_ThroughHole:SW_PUSH_SMALL
- U101: value PRTR5V0U4D -> AOZ8904; footprint (none) -> TO_SOT_Packages_SMD:SOT-23-6_Handsoldering; symbol PRTR5V0U4D -> AOZ8904; MPN (none) -> AOZ8904CIL
- U102: footprint (none) -> TO_SOT_Packages_SMD:TO-252-2Lead
- U103: footprint (none) -> Housings_QFP:LQFP-64_10x10mm_Pitch0.5mm
- U104: footprint (none) -> Housings_SOIC:SOIC-8_3.9x4.9mm_Pitch1.27mm
- Y101: footprint (none) -> Crystals:Crystal_HC49-U_Vertical
Connections:
- wire segments 118 -> 125
- no-connect marks 28 -> 25
Changed lines of the file:
@@
 F 0 "JP101" H 3890 2640 50  0000 C CNN
 F 1 "JUMPER" H 3890 2410 50  0000 C CNN
-F 2 "" H 3890 2490 50  0001 C CNN
+F 2 "stmps:MADW__SMD-solder-bridge-narrow" H 3890 2490 50  0001 C CNN
 F 3 "" H 3890 2490 50  0000 C CNN
 	1    3890 2490
@@
 $EndComp
 $Comp
-L CP_Small C114
+L C_Small C114
 U 1 1 579D543E
 P 4300 1550
 F 0 "C114" H 4325 1650 50  0000 L CNN
 F 1 "4.7uf" H 4325 1450 50  0000 L CNN
-F 2 "" H 4338 1400 50  0001 C CNN
+F 2 "Capacitors_SMD:C_0805_HandSoldering" H 4338 1400 50  0001 C CNN
 F 3 "" H 4300 1550 50  0000 C CNN
 	1    4300 1550
@@
 $EndComp
 $Comp
-L CP_Small C109
+L C_Small C109
 U 1 1 579D6E02
 P 3530 3110
 F 0 "C109" H 3555 3210 50  0000 L CNN
 F 1 "1uf" H 3555 3010 50  0000 L CNN
-F 2 "" H 3568 2960 50  0001 C CNN
+F 2 "Capacitors_SMD:C_0805_HandSoldering" H 3568 2960 50  0001 C CNN
 F 3 "" H 3530 3110 50  0000 C CNN
 	1    3530 3110
@@
 F 0 "U103" H 5040 2340 50  0000 L BNN
 F 1 "STM32F411RCTx" H 5400 5150 50  0000 R BNN
-F 2 "" H 5240 5140 50  0001 R TNN
+F 2 "Housings_QFP:LQFP-64_10x10mm_Pitch0.5mm" H 5240 5140 50  0001 R TNN
 F 3 "" H 5750 3900 50  0000 C CNN
 	1    5750 3900
@@
 F 0 "Y101" H 2730 3740 50  0000 C CNN
 F 1 "Crystal" H 2730 3440 50  0000 C CNN
-F 2 "" H 2730 3590 50  0001 C CNN
+F 2 "Crystals:Crystal_HC49-U_Vertical" H 2730 3590 50  0001 C CNN
 F 3 "" H 2730 3590 50  0000 C CNN
 F 4 "ABL-8.000MHZ-B2" H 2730 3590 60  0001 C CNN "MPN"
@@
 F 0 "U102" H 2420 1210 60  0000 C CNN
 F 1 "LM1117-3.3v" H 2270 1640 60  0000 C CNN
-F 2 "" H 2260 1470 60  0001 C CNN
+F 2 "TO_SOT_Packages_SMD:TO-252-2Lead" H 2260 1470 60  0001 C CNN
 F 3 "" H 2260 1470 60  0000 C CNN
 	1    2260 1430
@@
 $EndComp
 $Comp
-L CONN_02X02 P101
+L CONN_01X04 P101
 U 1 1 579F286B
-P 1290 2060
-F 0 "P101" H 1290 2210 50  0000 C CNN
-F 1 "12v IN" H 1290 1910 50  0000 C CNN
-F 2 "" H 1290 860 50  0001 C CNN
-F 3 "" H 1290 860 50  0000 C CNN
-	1    1290 2060
-	0    1    1    0
+P 1480 3610
+F 0 "P101" H 1480 3860 50  0000 C CNN
+F 1 "12v IN" V 1570 3620 50  0000 C CNN
+F 2 "stmps:5EHDRC_1x04" H 1480 2410 50  0001 C CNN
+F 3 "" H 1480 2410 50  0000 C CNN
+	1    1480 3610
+	1    0    0    -1
 $EndComp
 $Comp
 L GND #PWR06
 U 1 1 579F3070
-P 1290 2470
-F 0 "#PWR06" H 1290 2220 50  0001 C CNN
-F 1 "GND" H 1290 2320 50  0000 C CNN
-F 2 "" H 1290 2470 50  0000 C CNN
-F 3 "" H 1290 2470 50  0000 C CNN
-	1    1290 2470
+P 1100 3930
+F 0 "#PWR06" H 1100 3680 50  0001 C CNN
+F 1 "GND" H 1100 3780 50  0000 C CNN
+F 2 "" H 1100 3930 50  0000 C CNN
+F 3 "" H 1100 3930 50  0000 C CNN
+	1    1100 3930
 	0    -1   -1   0
 $EndComp
-Text GLabel 1340 1810 1    60   Input ~ 0
+Text GLabel 1150 3210 1    60   Input ~ 0
 +12v
-Text GLabel 1240 1810 1    60   Input ~ 0
+Text GLabel 1050 3210 1    60   Input ~ 0
 +12v-2
 Text GLabel 5000 1390 1    60   Input ~ 0
@@
 	4940 6010 5340 6010
 Wire Wire Line
-	1240 2320 1340 2320
-Wire Wire Line
-	1340 2320 1340 2310
-Wire Wire Line
-	1240 2320 1240 2310
-Wire Wire Line
-	1290 2320 1290 2650
-Connection ~ 1290 2320
-Wire Wire Line
 	1610 1390 1960 1390
 Wire Wire Line
@@
 L CONN_02X03 P102
 U 1 1 57A1EB2A
-P 1290 2900
-F 0 "P102" H 1290 3100 50  0000 C CNN
-F 1 "12v" H 1290 2700 50  0000 C CNN
-F 2 "" H 1290 1700 50  0001 C CNN
-F 3 "" H 1290 1700 50  0000 C CNN
-	1    1290 2900
+P 1100 4360
+F 0 "P102" H 1100 4560 50  0000 C CNN
+F 1 "12v" H 1100 4160 50  0000 C CNN
+F 2 "Pin_Headers:Pin_Header_Straight_2x03" H 1100 3160 50  0001 C CNN
+F 3 "" H 1100 3160 50  0000 C CNN
+	1    1100 4360
 	0    1    -1   0
 $EndComp
 Wire Wire Line
-	1190 2650 1190 2600
-Wire Wire Line
-	1190 2600 1390 2600
-Connection ~ 1290 2600
-Wire Wire Line
-	1390 2600 1390 2650
-Connection ~ 1290 2470
-Text GLabel 1290 3240 3    60   Input ~ 0
+	1000 4110 1000 4060
+Wire Wire Line
+	1000 4060 1200 4060
+Connection ~ 1100 4060
+Wire Wire Line
+	1200 4060 1200 4110
+Text GLabel 1100 4700 3    60   Input ~ 0
 +12v
 Wire Wire Line
-	1190 3150 1190 3240
-Wire Wire Line
-	1190 3240 1390 3240
-Wire Wire Line
-	1290 3240 1290 3150
-Wire Wire Line
-	1390 3240 1390 3150
-Connection ~ 1290 3240
+	1000 4610 1000 4700
+Wire Wire Line
+	1000 4700 1200 4700
+Wire Wire Line
+	1100 4700 1100 4610
+Wire Wire Line
+	1200 4700 1200 4610
+Connection ~ 1100 4700
 $Sheet
 S 8420 1490 870  750
@@
 F 0 "P103" H 2555 2025 50  0000 C CNN
 F 1 "USB_OTG" H 2230 2350 50  0000 C CNN
-F 2 "" V 2180 2050 50  0001 C CNN
+F 2 "Connect:USB_Micro-B" V 2180 2050 50  0001 C CNN
 F 3 "" V 2180 2050 50  0000 C CNN
 	1    2230 2150
@@
 NoConn ~ 2330 2450
 $Comp
-L PRTR5V0U4D U101
+L AOZ8904 U101
 U 1 1 57A62CBA
 P 2000 3060
 F 0 "U101" H 2160 2850 60  0000 C CNN
-F 1 "PRTR5V0U4D" H 2010 3280 60  0000 C CNN
-F 2 "" H 2000 3100 60  0001 C CNN
+F 1 "AOZ8904" H 2010 3280 60  0000 C CNN
+F 2 "TO_SOT_Packages_SMD:SOT-23-6_Handsoldering" H 2000 3100 60  0001 C CNN
 F 3 "" H 2000 3100 60  0000 C CNN
+F 4 "AOZ8904CIL" H 2000 3060 60  0001 C CNN "MPN"
 	1    2000 3060
 	1    0    0    -1
@@
 F 0 "C101" H 945 1580 50  0000 L CNN
 F 1 "100uf" H 945 1380 50  0000 L CNN
-F 2 "" H 958 1330 50  0001 C CNN
+F 2 "Capacitors_SMD:c_elec_6.3x5.8" H 958 1330 50  0001 C CNN
 F 3 "" H 920 1480 50  0000 C CNN
+F 4 "35TZV100M6.3X8" H 920 1480 60  0001 C CNN "MPN"
 	1    920  1480
 	1    0    0    -1
@@
 F 0 "U104" H 7410 6150 50  0000 C CNN
 F 1 "M24C04" H 7460 5450 50  0000 C CNN
-F 2 "" H 7260 5800 50  0001 C CNN
+F 2 "Housings_SOIC:SOIC-8_3.9x4.9mm_Pitch1.27mm" H 7260 5800 50  0001 C CNN
 F 3 "" H 7260 5800 50  0000 C CNN
 F 4 "M24C04-WMN6TP" H 7260 5800 60  0001 C CNN "MPN"
@@
 	1    0    0    -1
 $EndComp
-NoConn ~ 6560 5600
-NoConn ~ 6560 5700
-NoConn ~ 6560 5800
-Text GLabel 7260 5300 0    60   Input ~ 0
+Text GLabel 7130 5220 0    60   Input ~ 0
 +3.3v
 $Comp
@@
 F 0 "SW101" H 6680 4040 50  0000 C CNN
 F 1 "RST" H 6500 3930 50  0000 C CNN
-F 2 "" H 6560 3970 50  0001 C CNN
+F 2 "Buttons_Switches_ThroughHole:SW_PUSH_SMALL" H 6560 3970 50  0001 C CNN
 F 3 "" H 6560 3970 50  0000 C CNN
 	1    6560 3970
@@
 U 1 1 57AD4D95
 P 6340 3970
-F 0 "C115" H 6300 4060 50  0000 L CNN
-F 1 "0.1uf" V 6450 3900 50  0000 L CNN
+F 0 "C115" H 6250 3800 50  0000 L CNN
+F 1 "0.1uf" V 6450 3930 50  0000 L CNN
 F 2 "Capacitors_SMD:C_0805_HandSoldering" H 6378 3820 50  0001 C CNN
 F 3 "" H 6340 3970 50  0000 C CNN
@@
 L +12V #PWR019
 U 1 1 57AE7CE4
-P 1240 1840
-F 0 "#PWR019" H 1240 1690 50  0001 C CNN
-F 1 "+12V" H 1240 1980 50  0000 C CNN
-F 2 "" H 1240 1840 50  0000 C CNN
-F 3 "" H 1240 1840 50  0000 C CNN
-	1    1240 1840
+P 1050 3300
+F 0 "#PWR019" H 1050 3150 50  0001 C CNN
+F 1 "+12V" H 1050 3440 50  0000 C CNN
+F 2 "" H 1050 3300 50  0000 C CNN
+F 3 "" H 1050 3300 50  0000 C CNN
+	1    1050 3300
 	0    -1   -1   0
 $EndComp
@@
 L +12V #PWR020
 U 1 1 57AE7E36
-P 1340 1840
-F 0 "#PWR020" H 1340 1690 50  0001 C CNN
-F 1 "+12V" H 1340 1980 50  0000 C CNN
-F 2 "" H 1340 1840 50  0000 C CNN
-F 3 "" H 1340 1840 50  0000 C CNN
-	1    1340 1840
-	0    1    1    0
-$EndComp
-Connection ~ 1240 1840
-Connection ~ 1340 1840
+P 1150 3300
+F 0 "#PWR020" H 1150 3150 50  0001 C CNN
+F 1 "+12V" H 1150 3440 50  0000 C CNN
+F 2 "" H 1150 3300 50  0000 C CNN
+F 3 "" H 1150 3300 50  0000 C CNN
+	1    1150 3300
+	0    1    1    0
+$EndComp
 NoConn ~ 5800 2510
 NoConn ~ 5800 2610
@@
 Wire Wire Line
 	3650 2490 3790 2490
+Wire Wire Line
+	6560 6280 7260 6280
+Wire Wire Line
+	6560 5600 6560 6280
+Connection ~ 6560 5800
+Connection ~ 6560 5700
+Connection ~ 7260 6280
+$Comp
+L C_Small C118
+U 1 1 57B1C4CB
+P 7360 5220
+F 0 "C118" V 7260 5120 50  0000 L CNN
+F 1 "0.1uf" V 7470 5150 50  0000 L CNN
+F 2 "Capacitors_SMD:C_0805_HandSoldering" H 7398 5070 50  0001 C CNN
+F 3 "" H 7360 5220 50  0000 C CNN
+	1    7360 5220
+	0    1    1    0
+$EndComp
+$Comp
+L GND #PWR021
+U 1 1 57B1DB71
+P 7460 5220
+F 0 "#PWR021" H 7460 4970 50  0001 C CNN
+F 1 "GND" H 7460 5070 50  0000 C CNN
+F 2 "" H 7460 5220 50  0000 C CNN
+F 3 "" H 7460 5220 50  0000 C CNN
+	1    7460 5220
+	0    -1   -1   0
+$EndComp
+Wire Wire Line
+	7130 5220 7260 5220
+Wire Wire Line
+	7260 5220 7260 5300
+Connection ~ 7260 5220
+Wire Wire Line
+	1050 3210 1050 3660
+Wire Wire Line
+	1050 3660 1280 3660
+Wire Wire Line
+	1280 3460 1150 3460
+Wire Wire Line
+	1150 3460 1150 3210
+Connection ~ 1150 3300
+Connection ~ 1050 3300
+Wire Wire Line
+	1100 4110 1100 3560
+Wire Wire Line
+	1100 3560 1280 3560
+Wire Wire Line
+	1280 3760 1100 3760
+Connection ~ 1100 3760
+Connection ~ 1100 3930
 $EndSCHEMATC

Commit message: Complete routing, first pass.
Parts:
- removed C115: 0.1uf, Capacitors_SMD:C_0805_HandSoldering, symbol C_Small
- removed SW101: RST, Buttons_Switches_ThroughHole:SW_PUSH_SMALL, symbol SW_PUSH_SMALL
- removed W101, W102, W103, W104: TEST_1P, Connect:PINTST, symbol TEST_1P
- JP101: value JUMPER -> BOOT0; footprint stmps:MADW__SMD-solder-bridge-narrow -> Pin_Headers:Pin_Header_Straight_1x02_Pitch2.00mm; symbol Jumper_NC_Small -> CONN_01X02
Connections:
- net labels added: +5v
- net labels removed: +12v-2
- wire segments 125 -> 122
- no-connect marks 25 -> 29
Changed lines of the file:
@@
 $EndDescr
 $Comp
-L Jumper_NC_Small JP101
+L CONN_01X02 JP101
 U 1 1 579D4D3A
-P 3890 2490
-F 0 "JP101" H 3890 2640 50  0000 C CNN
-F 1 "JUMPER" H 3890 2410 50  0000 C CNN
-F 2 "stmps:MADW__SMD-solder-bridge-narrow" H 3890 2490 50  0001 C CNN
-F 3 "" H 3890 2490 50  0000 C CNN
-	1    3890 2490
-	1    0    0    -1
+P 3900 2290
+F 0 "JP101" H 3900 2440 50  0000 C CNN
+F 1 "BOOT0" H 3900 2210 50  0000 C CNN
+F 2 "Pin_Headers:Pin_Header_Straight_1x02_Pitch2.00mm" H 3900 2290 50  0001 C CNN
+F 3 "" H 3900 2290 50  0000 C CNN
+	1    3900 2290
+	0    -1   -1   0
 $EndComp
 $Comp
@@
 	0    -1   -1   0
 $EndComp
-Text GLabel 1150 3210 1    60   Input ~ 0
+Text GLabel 1100 3210 1    60   Input ~ 0
 +12v
-Text GLabel 1050 3210 1    60   Input ~ 0
-+12v-2
 Text GLabel 5000 1390 1    60   Input ~ 0
 +3.3v
@@
 Text Label 4460 5030 2    60   ~ 0
 Z_STEP
+Text Label 5810 5410 0    60   ~ 0
+E0_ENABLE
 Text Label 5810 5210 0    60   ~ 0
-E0_ENABLE
+E0_STEP
 Text Label 5810 5310 0    60   ~ 0
-E0_STEP
-Text Label 5810 5410 0    60   ~ 0
 E0_DIR
 Text Label 6330 3610 0    60   ~ 0
 SWDIO
 Wire Wire Line
-	3990 2490 4460 2490
+	3950 2490 4460 2490
 Wire Wire Line
 	4300 1650 4300 1830
@@
 Text GLabel 8420 2690 0    60   Input ~ 0
 +12v
-Text GLabel 8410 3600 0    60   Input ~ 0
-+12v-2
 Text Label 5800 3110 0    60   ~ 0
 FAN_PWM
@@
 	1680 2960 1680 2450
 Connection ~ 1680 2450
-Text Label 2320 3050 0    60   ~ 0
+Text Label 1680 3150 2    60   ~ 0
 USB_DN
-Text Label 2320 3150 0    60   ~ 0
+Text Label 1680 3050 2    60   ~ 0
 USB_DP
-NoConn ~ 1680 3050
-NoConn ~ 1680 3150
+NoConn ~ 2320 3050
+NoConn ~ 2320 3150
 Wire Wire Line
 	2320 2960 2550 2960
@@
 SDA
 $Comp
-L SW_PUSH_SMALL SW101
-U 1 1 57AD1454
-P 6560 3970
-F 0 "SW101" H 6680 4040 50  0000 C CNN
-F 1 "RST" H 6500 3930 50  0000 C CNN
-F 2 "Buttons_Switches_ThroughHole:SW_PUSH_SMALL" H 6560 3970 50  0001 C CNN
-F 3 "" H 6560 3970 50  0000 C CNN
-	1    6560 3970
-	1    0    0    -1
-$EndComp
-Wire Wire Line
-	6180 3870 6460 3870
-Connection ~ 6180 3870
-$Comp
-L C_Small C115
-U 1 1 57AD4D95
-P 6340 3970
-F 0 "C115" H 6250 3800 50  0000 L CNN
-F 1 "0.1uf" V 6450 3930 50  0000 L CNN
-F 2 "Capacitors_SMD:C_0805_HandSoldering" H 6378 3820 50  0001 C CNN
-F 3 "" H 6340 3970 50  0000 C CNN
-	1    6340 3970
-	-1   0    0    1
-$EndComp
-Connection ~ 6340 3870
-Wire Wire Line
-	6340 4070 6340 4210
-Wire Wire Line
-	6340 4210 6660 4210
-Wire Wire Line
-	6660 4210 6660 4070
-$Comp
-L GND #PWR018
-U 1 1 57AD539C
-P 6460 4210
-F 0 "#PWR018" H 6460 3960 50  0001 C CNN
-F 1 "GND" H 6460 4060 50  0000 C CNN
-F 2 "" H 6460 4210 50  0000 C CNN
-F 3 "" H 6460 4210 50  0000 C CNN
-	1    6460 4210
-	1    0    0    -1
-$EndComp
-Connection ~ 6460 4210
-$Comp
-L TEST_1P W104
-U 1 1 57ADEC1C
-P 9840 5640
-F 0 "W104" H 9840 5910 50  0000 C CNN
-F 1 "TEST_1P" H 9840 5840 50  0000 C CNN
-F 2 "Connect:PINTST" H 10040 5640 50  0001 C CNN
-F 3 "" H 10040 5640 50  0000 C CNN
-	1    9840 5640
-	0    -1   -1   0
-$EndComp
-$Comp
-L TEST_1P W102
-U 1 1 57ADF1E5
-P 9830 4030
-F 0 "W102" H 9830 4300 50  0000 C CNN
-F 1 "TEST_1P" H 9830 4230 50  0000 C CNN
-F 2 "Connect:PINTST" H 10030 4030 50  0001 C CNN
-F 3 "" H 10030 4030 50  0000 C CNN
-	1    9830 4030
-	0    -1   -1   0
-$EndComp
-$Comp
-L TEST_1P W103
-U 1 1 57AE07C2
-P 9840 3090
-F 0 "W103" H 9840 3360 50  0000 C CNN
-F 1 "TEST_1P" H 9840 3290 50  0000 C CNN
-F 2 "Connect:PINTST" H 10040 3090 50  0001 C CNN
-F 3 "" H 10040 3090 50  0000 C CNN
-	1    9840 3090
-	0    -1   -1   0
-$EndComp
-$Comp
-L TEST_1P W101
-U 1 1 57AE0942
-P 9830 2130
-F 0 "W101" H 9830 2400 50  0000 C CNN
-F 1 "TEST_1P" H 9830 2330 50  0000 C CNN
-F 2 "Connect:PINTST" H 10030 2130 50  0001 C CNN
-F 3 "" H 10030 2130 50  0000 C CNN
-	1    9830 2130
-	0    -1   -1   0
-$EndComp
-$Comp
-L +12V #PWR019
-U 1 1 57AE7CE4
+L +12V #PWR018
+U 1 1 57AE7E36
 P 1050 3300
-F 0 "#PWR019" H 1050 3150 50  0001 C CNN
+F 0 "#PWR018" H 1050 3150 50  0001 C CNN
 F 1 "+12V" H 1050 3440 50  0000 C CNN
 F 2 "" H 1050 3300 50  0000 C CNN
@@
 	1    1050 3300
 	0    -1   -1   0
-$EndComp
-$Comp
-L +12V #PWR020
-U 1 1 57AE7E36
-P 1150 3300
-F 0 "#PWR020" H 1150 3150 50  0001 C CNN
-F 1 "+12V" H 1150 3440 50  0000 C CNN
-F 2 "" H 1150 3300 50  0000 C CNN
-F 3 "" H 1150 3300 50  0000 C CNN
-	1    1150 3300
-	0    1    1    0
 $EndComp
 NoConn ~ 5800 2510
@@
 NoConn ~ 4460 4630
 Wire Wire Line
-	3650 2490 3790 2490
+	3650 2490 3850 2490
 Wire Wire Line
 	6560 6280 7260 6280
@@
 $EndComp
 $Comp
-L GND #PWR021
+L GND #PWR019
 U 1 1 57B1DB71
 P 7460 5220
-F 0 "#PWR021" H 7460 4970 50  0001 C CNN
+F 0 "#PWR019" H 7460 4970 50  0001 C CNN
 F 1 "GND" H 7460 5070 50  0000 C CNN
 F 2 "" H 7460 5220 50  0000 C CNN
@@
 Connection ~ 1100 3760
 Connection ~ 1100 3930
+NoConn ~ 9840 5640
+NoConn ~ 9830 4030
+NoConn ~ 9840 3090
+NoConn ~ 9830 2130
+Text Label 1610 1910 0    60   ~ 0
++5v
+Wire Wire Line
+	1150 3210 1050 3210
+Text GLabel 8410 3600 0    60   Input ~ 0
++12v
 $EndSCHEMATC

Commit message: Finalized layout for Alpha 1.
Parts:
- U103: MPN (none) -> STM32F411RCT6
Changed lines of the file:
@@
 F 2 "Housings_QFP:LQFP-64_10x10mm_Pitch0.5mm" H 5240 5140 50  0001 R TNN
 F 3 "" H 5750 3900 50  0000 C CNN
+F 4 "STM32F411RCT6" H 5750 3900 60  0001 C CNN "MPN"
 	1    5750 3900
 	1    0    0    -1

Commit message: Fix USB connection. Cleanups.
Connections:
- net labels added: USB_DM
- net labels removed: USB_DN
- wire segments 122 -> 129
Other:
- note added: "DP may need a pullup"
Changed lines of the file:
@@
 $EndComp
 Text Label 5800 3410 0    60   ~ 0
+USB_DM
+Text Label 5800 3510 0    60   ~ 0
 USB_DP
-Text Label 5800 3510 0    60   ~ 0
-USB_DN
 $Comp
 L USB_OTG P103
@@
 $EndComp
 Connection ~ 2630 2230
-Text Label 2230 2450 3    60   ~ 0
-USB_DP
-Text Label 2130 2450 3    60   ~ 0
-USB_DN
-Wire Wire Line
-	1610 1390 1610 2450
 Wire Wire Line
 	1610 2450 2030 2450
 NoConn ~ 2330 2450
-$Comp
-L AOZ8904 U101
-U 1 1 57A62CBA
-P 2000 3060
-F 0 "U101" H 2160 2850 60  0000 C CNN
-F 1 "AOZ8904" H 2010 3280 60  0000 C CNN
-F 2 "TO_SOT_Packages_SMD:SOT-23-6_Handsoldering" H 2000 3100 60  0001 C CNN
-F 3 "" H 2000 3100 60  0000 C CNN
-F 4 "AOZ8904CIL" H 2000 3060 60  0001 C CNN "MPN"
-	1    2000 3060
-	1    0    0    -1
-$EndComp
-Wire Wire Line
-	1680 2960 1680 2450
-Connection ~ 1680 2450
-Text Label 1680 3150 2    60   ~ 0
-USB_DN
-Text Label 1680 3050 2    60   ~ 0
+Text Label 2090 2630 2    60   ~ 0
+USB_DM
+Text Label 2320 2620 0    60   ~ 0
 USB_DP
-NoConn ~ 2320 3050
-NoConn ~ 2320 3150
-Wire Wire Line
-	2320 2960 2550 2960
-Wire Wire Line
-	2550 2960 2550 2450
-Connection ~ 2550 2450
 $Comp
 L C_Small C106
@@
 	1050 3660 1280 3660
 Wire Wire Line
-	1280 3460 1150 3460
-Wire Wire Line
-	1150 3460 1150 3210
+	1150 3460 1280 3460
+Wire Wire Line
+	1150 3210 1150 3460
 Connection ~ 1150 3300
 Connection ~ 1050 3300
 Wire Wire Line
-	1100 4110 1100 3560
+	1100 3560 1100 4110
 Wire Wire Line
 	1100 3560 1280 3560
@@
 Text GLabel 8410 3600 0    60   Input ~ 0
 +12v
+Text Notes 2440 2730 0    60   ~ 0
+DP may need a pullup
+$Comp
+L AOZ8904 U101
+U 1 1 57A62CBA
+P 2220 3030
+F 0 "U101" H 2120 2830 60  0000 C CNN
+F 1 "AOZ8904" H 2230 3250 60  0000 C CNN
+F 2 "TO_SOT_Packages_SMD:SOT-23-6_Handsoldering" H 2220 3070 60  0001 C CNN
+F 3 "" H 2220 3070 60  0000 C CNN
+F 4 "AOZ8904CIL" H 2220 3030 60  0001 C CNN "MPN"
+	1    2220 3030
+	1    0    0    -1
+$EndComp
+Wire Wire Line
+	1610 1390 1610 2930
+Wire Wire Line
+	2230 2450 2230 2620
+Wire Wire Line
+	2230 2620 2820 2620
+Wire Wire Line
+	2820 2620 2820 3020
+Wire Wire Line
+	2820 3020 2540 3020
+Wire Wire Line
+	2130 2450 2130 2630
+Wire Wire Line
+	2130 2630 1730 2630
+Wire Wire Line
+	1730 2630 1730 3120
+Wire Wire Line
+	1730 3120 1900 3120
+Wire Wire Line
+	1610 2930 1900 2930
+Connection ~ 1610 2450
+$Comp
+L GND #PWR?
+U 1 1 57A7DE49
+P 2580 2930
+F 0 "#PWR?" H 2580 2680 50  0001 C CNN
+F 1 "GND" H 2580 2780 50  0000 C CNN
+F 2 "" H 2580 2930 50  0000 C CNN
+F 3 "" H 2580 2930 50  0000 C CNN
+	1    2580 2930
+	0    -1   -1   0
+$EndComp
+Wire Wire Line
+	2540 2930 2580 2930
+NoConn ~ 2540 3120
+NoConn ~ 1900 3020
 $EndSCHEMATC

Commit message: WIP rev B.
Parts:
- removed C118: 0.1uf, Capacitors_SMD:C_0805_HandSoldering, symbol C_Small
- removed R107, R108: 4.7k, Resistors_SMD:R_0805_HandSoldering, symbol R_Small
- removed U104: M24C04, Housings_SOIC:SOIC-8_3.9x4.9mm_Pitch1.27mm, symbol 24C16
- added D103: D_Schottky_Small, Diodes_SMD:SOD-123, symbol D_Schottky_Small
- added U105: CHIP-TOP, stmps:CHIP-MIN, symbol CHIP-TOP
Connections:
- net labels added: CHIP_1_WIRE, USART1_RX, USART1_TX
- wire segments 129 -> 128
- no-connect marks 29 -> 25
