File: high_power_fet.sch (KiCad schematic (older format))
At the start: 6 parts, among them P701 OUT, Q701 IPP039N04L

Commit message: Start working on footprint assignments.
Parts:
- D701: footprint (none) -> LEDs:LED_0805
- P701: footprint (none) -> Pin_Headers:Pin_Header_Straight_1x02
- R701, R702, R703: footprint (none) -> Resistors_SMD:R_0805_HandSoldering
Changed lines of the file:
@@
 F 0 "R801" H 5470 4250 50  0000 L CNN
 F 1 "100k" H 5470 4190 50  0000 L CNN
-F 2 "" H 5440 4230 50  0000 C CNN
+F 2 "Resistors_SMD:R_0805_HandSoldering" H 5440 4230 50  0001 C CNN
 F 3 "" H 5440 4230 50  0000 C CNN
 	1    5440 4230
@@
 F 0 "P801" H 6400 3570 50  0000 C CNN
 F 1 "OUT" V 6500 3420 50  0000 C CNN
-F 2 "" H 6400 3420 50  0000 C CNN
+F 2 "Pin_Headers:Pin_Header_Straight_1x02" H 6400 3420 50  0001 C CNN
 F 3 "" H 6400 3420 50  0000 C CNN
 	1    6400 3420
@@
 F 0 "R802" V 5730 3940 50  0000 L CNN
 F 1 "100" V 5600 3900 50  0000 L CNN
-F 2 "" H 5660 3980 50  0000 C CNN
+F 2 "Resistors_SMD:R_0805_HandSoldering" H 5660 3980 50  0001 C CNN
 F 3 "" H 5660 3980 50  0000 C CNN
 	1    5660 3980
@@
 F 0 "Q801" H 6260 4030 50  0000 R CNN
 F 1 "IPP039N04L" H 5940 4120 50  0000 R CNN
-F 2 "" H 6160 4080 50  0000 C CNN
+F 2 "" H 6160 4080 50  0001 C CNN
 F 3 "" H 5960 3980 50  0000 C CNN
 F 4 "IPP039N04LGXKSA1-ND" H 5960 3980 60  0001 C CNN "MPN"
@@
 F 0 "R803" V 6010 3470 50  0000 L CNN
 F 1 "560" V 5880 3430 50  0000 L CNN
-F 2 "" H 5940 3510 50  0000 C CNN
+F 2 "Resistors_SMD:R_0805_HandSoldering" H 5940 3510 50  0001 C CNN
 F 3 "" H 5940 3510 50  0000 C CNN
 	1    5940 3510
@@
 F 0 "D801" H 6070 3760 50  0000 L CNN
 F 1 "r" H 5885 3560 50  0001 L CNN
-F 2 "" V 6060 3660 50  0000 C CNN
+F 2 "LEDs:LED_0805" V 6060 3660 50  0001 C CNN
 F 3 "" V 6060 3660 50  0000 C CNN
 	1    6060 3660

Commit message: Finish assigning footprints.
Parts:
- P701: footprint Pin_Headers:Pin_Header_Straight_1x02 -> stmps:TB-1x02
- Q701: footprint (none) -> TO_SOT_Packages_THT:TO-220_Neutral123_Vertical
Changed lines of the file:
@@
 $Descr A4 11693 8268
 encoding utf-8
-Sheet 8 8
+Sheet 7 8
 Title ""
 Date ""
@@
 $EndDescr
 $Comp
-L GND #PWR030
+L GND #PWR031
 U 1 1 57A29750
 P 6190 4330
-AR Path="/57A291CF/57A29750" Ref="#PWR030"  Part="1"
-AR Path="/57A2D9CC/57A29750" Ref="#PWR031"  Part="1"
-F 0 "#PWR031" H 6190 4080 50  0001 C CNN
+AR Path="/57A291CF/57A29750" Ref="#PWR031"  Part="1"
+AR Path="/57A2D9CC/57A29750" Ref="#PWR032"  Part="1"
+F 0 "#PWR032" H 6190 4080 50  0001 C CNN
 F 1 "GND" H 6190 4180 50  0000 C CNN
 F 2 "" H 6190 4330 50  0000 C CNN
@@
 F 0 "P801" H 6400 3570 50  0000 C CNN
 F 1 "OUT" V 6500 3420 50  0000 C CNN
-F 2 "Pin_Headers:Pin_Header_Straight_1x02" H 6400 3420 50  0001 C CNN
+F 2 "stmps:TB-1x02" H 6400 3420 50  0001 C CNN
 F 3 "" H 6400 3420 50  0000 C CNN
 	1    6400 3420
@@
 F 0 "Q801" H 6260 4030 50  0000 R CNN
 F 1 "IPP039N04L" H 5940 4120 50  0000 R CNN
-F 2 "" H 6160 4080 50  0001 C CNN
+F 2 "TO_SOT_Packages_THT:TO-220_Neutral123_Vertical" H 6160 4080 50  0001 C CNN
 F 3 "" H 5960 3980 50  0000 C CNN
 F 4 "IPP039N04LGXKSA1-ND" H 5960 3980 60  0001 C CNN "MPN"

Commit message: Complete routing, first pass.
Parts:
- P701: footprint stmps:TB-1x02 -> Connectors_Molex:Molex_KK-6410-02_02x2.54mm_Straight
Changed lines of the file:
@@
 $EndDescr
 $Comp
-L GND #PWR031
+L GND #PWR029
 U 1 1 57A29750
 P 6190 4330
-AR Path="/57A291CF/57A29750" Ref="#PWR031"  Part="1"
-AR Path="/57A2D9CC/57A29750" Ref="#PWR032"  Part="1"
-F 0 "#PWR032" H 6190 4080 50  0001 C CNN
+AR Path="/57A291CF/57A29750" Ref="#PWR029"  Part="1"
+AR Path="/57A2D9CC/57A29750" Ref="#PWR030"  Part="1"
+F 0 "#PWR030" H 6190 4080 50  0001 C CNN
 F 1 "GND" H 6190 4180 50  0000 C CNN
 F 2 "" H 6190 4330 50  0000 C CNN
@@
 F 0 "P801" H 6400 3570 50  0000 C CNN
 F 1 "OUT" V 6500 3420 50  0000 C CNN
-F 2 "stmps:TB-1x02" H 6400 3420 50  0001 C CNN
+F 2 "Connectors_Molex:Molex_KK-6410-02_02x2.54mm_Straight" H 6400 3420 50  0001 C CNN
 F 3 "" H 6400 3420 50  0000 C CNN
 	1    6400 3420

Commit message: Fix USB connection. Cleanups.
Connections:
- wire segments 13 -> 14
Changed lines of the file:
@@
 $EndDescr
 $Comp
-L GND #PWR029
+L GND #PWR030
 U 1 1 57A29750
-P 6190 4330
-AR Path="/57A291CF/57A29750" Ref="#PWR029"  Part="1"
-AR Path="/57A2D9CC/57A29750" Ref="#PWR030"  Part="1"
-F 0 "#PWR030" H 6190 4080 50  0001 C CNN
-F 1 "GND" H 6190 4180 50  0000 C CNN
-F 2 "" H 6190 4330 50  0000 C CNN
-F 3 "" H 6190 4330 50  0000 C CNN
-	1    6190 4330
+P 5830 4330
+AR Path="/57A291CF/57A29750" Ref="#PWR030"  Part="1"
+AR Path="/57A2D9CC/57A29750" Ref="#PWR031"  Part="1"
+F 0 "#PWR031" H 5830 4080 50  0001 C CNN
+F 1 "GND" H 5830 4180 50  0000 C CNN
+F 2 "" H 5830 4330 50  0000 C CNN
+F 3 "" H 5830 4330 50  0000 C CNN
+	1    5830 4330
 	1    0    0    -1
 $EndComp
@@
 	6060 4180 6190 4180
 Wire Wire Line
-	6060 3780 6190 3780
+	6190 3780 6060 3780
 Wire Wire Line
-	6190 4180 6190 4330
-Wire Wire Line
-	6190 3780 6190 3470
+	6190 3470 6190 3780
 Wire Wire Line
 	6190 3470 6200 3470
@@
 L R_Small R701
 U 1 1 57A2976A
-P 5440 4230
+P 5440 4160
 AR Path="/57A291CF/57A2976A" Ref="R701"  Part="1"
 AR Path="/57A2D9CC/57A2976A" Ref="R801"  Part="1"
-F 0 "R801" H 5470 4250 50  0000 L CNN
-F 1 "100k" H 5470 4190 50  0000 L CNN
-F 2 "Resistors_SMD:R_0805_HandSoldering" H 5440 4230 50  0001 C CNN
-F 3 "" H 5440 4230 50  0000 C CNN
-	1    5440 4230
+F 0 "R701" H 5470 4180 50  0000 L CNN
+F 1 "100k" H 5470 4120 50  0000 L CNN
+F 2 "Resistors_SMD:R_0805_HandSoldering" H 5440 4160 50  0001 C CNN
+F 3 "" H 5440 4160 50  0000 C CNN
+	1    5440 4160
 	1    0    0    -1
 $EndComp
-Wire Wire Line
-	6190 4330 5440 4330
-Connection ~ 6190 4330
+Connection ~ 5830 4330
 $Comp
 L CONN_01X02 P701
@@
 AR Path="/57A291CF/57A29756" Ref="P701"  Part="1"
 AR Path="/57A2D9CC/57A29756" Ref="P801"  Part="1"
-F 0 "P801" H 6400 3570 50  0000 C CNN
+F 0 "P701" H 6400 3570 50  0000 C CNN
 F 1 "OUT" V 6500 3420 50  0000 C CNN
 F 2 "Connectors_Molex:Molex_KK-6410-02_02x2.54mm_Straight" H 6400 3420 50  0001 C CNN
@@
 $EndComp
 Wire Wire Line
-	5440 4130 5440 3980
+	5440 4060 5440 3980
 Wire Wire Line
 	5290 3980 5560 3980
@@
 AR Path="/57A291CF/57A2995A" Ref="R702"  Part="1"
 AR Path="/57A2D9CC/57A2995A" Ref="R802"  Part="1"
-F 0 "R802" V 5730 3940 50  0000 L CNN
+F 0 "R702" V 5730 3880 50  0000 L CNN
 F 1 "100" V 5600 3900 50  0000 L CNN
 F 2 "Resistors_SMD:R_0805_HandSoldering" H 5660 3980 50  0001 C CNN
@@
 AR Path="/57A291CF/57A29742" Ref="Q701"  Part="1"
 AR Path="/57A2D9CC/57A29742" Ref="Q801"  Part="1"
-F 0 "Q801" H 6260 4030 50  0000 R CNN
+F 0 "Q701" H 6310 4060 50  0000 R CNN
 F 1 "IPP039N04L" H 5940 4120 50  0000 R CNN
 F 2 "TO_SOT_Packages_THT:TO-220_Neutral123_Vertical" H 6160 4080 50  0001 C CNN
@@
 AR Path="/57A291CF/57A9EB82" Ref="R703"  Part="1"
 AR Path="/57A2D9CC/57A9EB82" Ref="R803"  Part="1"
-F 0 "R803" V 6010 3470 50  0000 L CNN
+F 0 "R703" V 6010 3410 50  0000 L CNN
 F 1 "560" V 5880 3430 50  0000 L CNN
 F 2 "Resistors_SMD:R_0805_HandSoldering" H 5940 3510 50  0001 C CNN
@@
 AR Path="/57A291CF/57A9EC55" Ref="D701"  Part="1"
 AR Path="/57A2D9CC/57A9EC55" Ref="D801"  Part="1"
-F 0 "D801" H 6070 3760 50  0000 L CNN
+F 0 "D701" H 6070 3760 50  0000 L CNN
 F 1 "r" H 5885 3560 50  0001 L CNN
 F 2 "LEDs:LED_0805" V 6060 3660 50  0001 C CNN
@@
 	6160 3660 6190 3660
 Connection ~ 6190 3660
+Wire Wire Line
+	5440 4260 5440 4330
+Wire Wire Line
+	5440 4330 6190 4330
+Wire Wire Line
+	6190 4330 6190 4180
 $EndSCHEMATC

Commit message: Alpha 3. Fix solder mask clearance. Fix 3.3v not tied to ref+. Tweaks and cleanups.
Parts:
- removed P701: OUT, Connectors_Molex:Molex_KK-6410-02_02x2.54mm_Straight, symbol CONN_01X02
Connections:
- net labels added: OUT+, OUT-
Changed lines of the file:
@@
 $Descr A4 11693 8268
 encoding utf-8
-Sheet 7 8
+Sheet 8 8
 Title ""
 Date ""
@@
 $EndComp
 Connection ~ 5830 4330
-$Comp
-L CONN_01X02 P701
-U 1 1 57A29756
-P 6400 3420
-AR Path="/57A291CF/57A29756" Ref="P701"  Part="1"
-AR Path="/57A2D9CC/57A29756" Ref="P801"  Part="1"
-F 0 "P801" H 6400 3570 50  0000 C CNN
-F 1 "OUT" V 6500 3420 50  0000 C CNN
-F 2 "Connectors_Molex:Molex_KK-6410-02_02x2.54mm_Straight" H 6400 3420 50  0001 C CNN
-F 3 "" H 6400 3420 50  0000 C CNN
-	1    6400 3420
-	1    0    0    -1
-$EndComp
 Wire Wire Line
 	5440 4060 5440 3980
@@
 Wire Wire Line
 	6190 4330 6190 4180
+Text HLabel 6200 3370 2    60   Input ~ 0
+OUT+
+Text HLabel 6200 3470 2    60   Input ~ 0
+OUT-
 $EndSCHEMATC

Commit message: Update stuff. ;)
Parts:
- D701: symbol Led_Small -> LED_Small
Changed lines of the file:
@@
 EESchema Schematic File Version 2
+LIBS:STMPS-rescue
 LIBS:power
 LIBS:device
@@
 LIBS:gl-power
 LIBS:stmps
-LIBS:STMPS-cache
 EELAYER 25 0
 EELAYER END
@@
 Connection ~ 5940 3370
 $Comp
-L Led_Small D701
+L LED_Small D701
 U 1 1 57A9EC55
 P 6060 3660
 AR Path="/57A291CF/57A9EC55" Ref="D701"  Part="1"
 AR Path="/57A2D9CC/57A9EC55" Ref="D801"  Part="1"
+AR Path="/57A9EC55" Ref="D801"  Part="1"
 F 0 "D801" H 6070 3760 50  0000 L CNN
 F 1 "r" H 5885 3560 50  0001 L CNN
