File: low_power_fet.sch (KiCad schematic (older format))
At the start: 4 parts, among them P601 OUT, Q601 SSM3K333

Commit message: Start working on footprint assignments.
Parts:
- P601: footprint (none) -> Pin_Headers:Pin_Header_Straight_1x02
- R601: footprint (none) -> Resistors_SMD:R_0805_HandSoldering
Changed lines of the file:
@@
 F 0 "Q601" H 6170 3970 50  0000 R CNN
 F 1 "SSM3K333" H 5850 4060 50  0000 R CNN
-F 2 "" H 6070 4020 50  0000 C CNN
+F 2 "" H 6070 4020 50  0001 C CNN
 F 3 "" H 5870 3920 50  0000 C CNN
 F 4 "SSM3K333RLFCT-ND" H 5870 3920 60  0001 C CNN "MPN"
@@
 F 0 "D601" H 6170 4010 50  0000 L CNN
 F 1 "D_Schottky_Small" H 5940 3850 50  0001 L CNN
-F 2 "" V 6220 3930 50  0000 C CNN
+F 2 "" V 6220 3930 50  0001 C CNN
 F 3 "" V 6220 3930 50  0000 C CNN
 	1    6220 3930
@@
 F 0 "P601" H 6310 3510 50  0000 C CNN
 F 1 "OUT" V 6410 3360 50  0000 C CNN
-F 2 "" H 6310 3360 50  0000 C CNN
+F 2 "Pin_Headers:Pin_Header_Straight_1x02" H 6310 3360 50  0001 C CNN
 F 3 "" H 6310 3360 50  0000 C CNN
 	1    6310 3360
@@
 F 0 "R601" H 5700 4190 50  0000 L CNN
 F 1 "100k" H 5700 4130 50  0000 L CNN
-F 2 "" H 5670 4170 50  0000 C CNN
+F 2 "Resistors_SMD:R_0805_HandSoldering" H 5670 4170 50  0001 C CNN
 F 3 "" H 5670 4170 50  0000 C CNN
 	1    5670 4170

Commit message: Finish assigning footprints.
Parts:
- D601: footprint (none) -> Diodes_SMD:SOD-123; MPN (none) -> DB2J41100L
- P601: value OUT -> LP_OUT
- Q601: footprint (none) -> TO_SOT_Packages_SMD:SOT-23_Handsoldering
Changed lines of the file:
@@
 F 0 "Q601" H 6170 3970 50  0000 R CNN
 F 1 "SSM3K333" H 5850 4060 50  0000 R CNN
-F 2 "" H 6070 4020 50  0001 C CNN
+F 2 "TO_SOT_Packages_SMD:SOT-23_Handsoldering" H 6070 4020 50  0001 C CNN
 F 3 "" H 5870 3920 50  0000 C CNN
 F 4 "SSM3K333RLFCT-ND" H 5870 3920 60  0001 C CNN "MPN"
@@
 F 0 "D601" H 6170 4010 50  0000 L CNN
 F 1 "D_Schottky_Small" H 5940 3850 50  0001 L CNN
-F 2 "" V 6220 3930 50  0001 C CNN
+F 2 "Diodes_SMD:SOD-123" V 6220 3930 50  0001 C CNN
 F 3 "" V 6220 3930 50  0000 C CNN
+F 4 "DB2J41100L" H 6220 3930 60  0001 C CNN "MPN"
 	1    6220 3930
 	0    1    1    0
 $EndComp
 $Comp
-L GND #PWR029
+L GND #PWR030
 U 1 1 57A2899A
 P 6100 4270
-F 0 "#PWR029" H 6100 4020 50  0001 C CNN
+F 0 "#PWR030" H 6100 4020 50  0001 C CNN
 F 1 "GND" H 6100 4120 50  0000 C CNN
 F 2 "" H 6100 4270 50  0000 C CNN
@@
 P 6310 3360
 F 0 "P601" H 6310 3510 50  0000 C CNN
-F 1 "OUT" V 6410 3360 50  0000 C CNN
+F 1 "LP_OUT" V 6410 3360 50  0000 C CNN
 F 2 "Pin_Headers:Pin_Header_Straight_1x02" H 6310 3360 50  0001 C CNN
 F 3 "" H 6310 3360 50  0000 C CNN
